File: NixieClock.sch (EAGLE design)
At the start: 30 parts, among them IC1 SN75468D, IC10 SN74HC595PW, IC2 SN75468D, IC3 SN75468D, IC4 SN75468D, IC5 SN74HC595PW, IC6 SN74HC595PW, IC7 SN74HC595PW, IC8 SN74HC595PW, IC9 SN75468D, Q1 NIXIE-IN-8-2, Q2 NIXIE-IN-8-2, Q3 NIXIE-IN-8-2, Q4 NIXIE-IN-8-2, U1 TM4C1231H6PMI7PM

Commit message: Update
Parts:
- added D2, D3, D4, D5: 91V, Diodes:MMSZ5270BT1G
- added R10, R11, R12, R13: 10k, Resistors:CRCW121010K0FK
- added R14, R15, R16, R17, R5: 1M, Resistors:CRCW06031M00FK
- R1: device Resistors:RES100-1%-0.1W-16081608 -> Resistors:CRCW0603100RFK
- R2, R3, R4: device Resistors:RES10K-1%-0.1W-16081608 -> Resistors:CRCW060310K0FK
- R6, R7, R8, R9: device Resistors:RES33-1%-0.1W-16081608 -> Resistors:CRCW060333R0FK
Connections:
- removed net N$67: IC10.QB, IC9.2B
- removed net N$68: IC10.QC, IC9.3B
- removed net N$69: IC10.QD, IC9.4B
- removed net N$70: IC10.QE, IC9.5B
- removed net N$71: IC10.QF, IC9.6B
- removed net N$72: IC10.QG, IC9.7B
- new net HV: R10.P$2, R11.P$2, R12.P$2, R13.P$2, R14.P$2, R15.P$2, R16.P$2, R17.P$2, R5.P$2
- new net N$55: Q1.A, R10.P$1
- new net N$74: Q2.A, R11.P$1
- new net N$75: Q3.A, R12.P$1
- new net N$76: Q4.A, R13.P$1
- new net N$77: D2.1, IC2.COM, R14.P$1
- new net N$78: D3.1, IC3.COM, R15.P$1
- new net N$79: D4.1, IC4.COM, R16.P$1
- new net N$80: D5.1, IC9.COM, R17.P$1
- net GND: now also D2.2, D3.2, D4.2, D5.2, IC9.2B, IC9.3B, IC9.4B, IC9.5B, IC9.6B, IC9.7B
- net N$56: now also R5.P$1

Commit message: Update
Parts:
- removed D2, D3, D4, D5: 91V, Diodes:MMSZ5270BT1G
- removed R15, R16, R17: 1M, Resistors:CRCW06031M00FK
- removed U$17: JTAG-10PIN-ARM-CONN, Connectors:JTAG-10PIN-ARM-CONN
- added C6: 3u3/25V, Capacitors:C2012X7R1E335K125
- added M1: JTAG-10PIN-ARM-CONN, Connectors:JTAG-10PIN-ARM-CONN
- C1, C2, C3, C4, C5: value 10n -> 10n/50V
- D1: value 91V -> 91V/5%
- R1: value 100 -> 100/1%
- R10, R11, R12, R13, R2, R3, R4: value 10k -> 10k/1%
- R14: value 1M -> 33/1%; device Resistors:CRCW06031M00FK -> Resistors:CRCW060333R0FK
- R5: value 1M -> 1M/1%
- R6, R7, R8, R9: value 33 -> 33/1%
- U1: value TM4C1231H6PMI7PM -> TM4C1231H6PMI7; device Nixie:TM4C1231H6PMI7PM -> Nixie:TM4C1231H6PMI7
Connections:
- removed net JTAG_RST_N: U$17.10/RST_N
- removed net N$77: D2.1, IC2.COM, R14.P$1
- removed net N$78: D3.1, IC3.COM, R15.P$1
- removed net N$79: D4.1, IC4.COM, R16.P$1
- removed net N$80: D5.1, IC9.COM, R17.P$1
- new net !JTAG_RST: R14.P$2, U1.!RST
- new net DTA_COM: D1.1, IC1.COM, IC2.COM, IC3.COM, IC4.COM, IC9.COM, R5.P$1
- new net N$36: IC1.5C, Q2.K1
- new net N$37: IC1.6C, Q2.K2
- new net U1_VDDC: C6.1, U1.VDDC, U1.VDDC_2
- net 3V3: now also U1.VDD, U1.VDDA, U1.VDD_2, U1.VDD_3, U1.VDD_4
- net GND: now also C6.2, M1.3/GND1, M1.5/GND2, M1.9/GND3, U1.GND, U1.GNDA, U1.GNDX, U1.GND_2, U1.GND_3, U1.GND_4; no longer D2.2, D3.2, D4.2, D5.2, U$17.3/GND1, U$17.5/GND2, U$17.9/GND3
- net HV: no longer R14.P$2, R15.P$2, R16.P$2, R17.P$2
- net N$35: no longer IC1.5C, IC1.6C, Q2.K1, Q2.K2
- net N$39: now also M1.1/VCC; no longer U$17.1/VCC
- net N$40: now also M1.2/TMS; no longer U$17.2/TMS
- net N$41: now also M1.4/TCK; no longer U$17.4/TCK
- net N$42: now also M1.6/TDO; no longer U$17.6/TDO
- net N$43: now also M1.8/TDI; no longer U$17.8/TDI
- net N$56: now also M1.!10/RST, R14.P$1; no longer D1.1, IC1.COM, R5.P$1
Other:
- moved on the sheet: D1, IC10, IC2, IC3, IC4, IC6, IC7, IC8, IC9, Q1, Q2, Q3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

Commit message: Update
Parts:
- added PS1: S8421-45R, Misc:S8421-45R
- IC1, IC2, IC3, IC4, IC9: device Nixie:SN75468D -> ICs:SN75468D
- IC10, IC5, IC6, IC7, IC8: device Nixie:SN74HC595PW -> ICs:SN74HC595PW
- Q1, Q2, Q3, Q4: device Nixie:NIXIE-IN-8-2 -> Misc:NIXIE-IN-8-2
- U1: device Nixie:TM4C1231H6PMI7 -> ICs:TM4C1231H6PMI7
Connections:
- new net VBAT: PS1.ANODE, U1.VBAT
- net GND: now also PS1.CATHODE
Other:
- moved on the sheet: C6
Changed lines of the file:
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@@
 </classes>
 <parts>
-<part name="IC1" library="Nixie" deviceset="SN75468" device="D" package3d_urn="urn:adsk.eagle:package:24873557/2"/>
-<part name="IC2" library="Nixie" deviceset="SN75468" device="D" package3d_urn="urn:adsk.eagle:package:24873557/2"/>
-<part name="IC3" library="Nixie" deviceset="SN75468" device="D" package3d_urn="urn:adsk.eagle:package:24873557/2"/>
-<part name="IC4" library="Nixie" deviceset="SN75468" device="D" package3d_urn="urn:adsk.eagle:package:24873557/2"/>
-<part name="IC5" library="Nixie" deviceset="SN74HC595" device="PW" package3d_urn="urn:adsk.eagle:package:24918114/2"/>
-<part name="IC6" library="Nixie" deviceset="SN74HC595" device="PW" package3d_urn="urn:adsk.eagle:package:24918114/2"/>
-<part name="IC7" library="Nixie" deviceset="SN74HC595" device="PW" package3d_urn="urn:adsk.eagle:package:24918114/2"/>
-<part name="IC8" library="Nixie" deviceset="SN74HC595" device="PW" package3d_urn="urn:adsk.eagle:package:24918114/2"/>
+<part name="IC1" library="ICs" deviceset="SN75468" device="D" package3d_urn="urn:adsk.eagle:package:24873557/2"/>
+<part name="IC2" library="ICs" deviceset="SN75468" device="D" package3d_urn="urn:adsk.eagle:package:24873557/2"/>
+<part name="IC3" library="ICs" deviceset="SN75468" device="D" package3d_urn="urn:adsk.eagle:package:24873557/2"/>
+<part name="IC4" library="ICs" deviceset="SN75468" device="D" package3d_urn="urn:adsk.eagle:package:24873557/2"/>
+<part name="IC5" library="ICs" deviceset="SN74HC595" device="PW" package3d_urn="urn:adsk.eagle:package:24918114/2"/>
+<part name="IC6" library="ICs" deviceset="SN74HC595" device="PW" package3d_urn="urn:adsk.eagle:package:24918114/2"/>
+<part name="IC7" library="ICs" deviceset="SN74HC595" device="PW" package3d_urn="urn:adsk.eagle:package:24918114/2"/>
+<part name="IC8" library="ICs" deviceset="SN74HC595" device="PW" package3d_urn="urn:adsk.eagle:package:24918114/2"/>
 <part name="C1" library="Capacitors" deviceset="C0603C103K5RACTU" device="" package3d_urn="urn:adsk.eagle:package:24972866/1" value="10n/50V"/>
 <part name="C2" library="Capacitors" deviceset="C0603C103K5RACTU" device="" package3d_urn="urn:adsk.eagle:package:24972866/1" value="10n/50V"/>
 <part name="C3" library="Capacitors" deviceset="C0603C103K5RACTU" device="" package3d_urn="urn:adsk.eagle:package:24972866/1" value="10n/50V"/>
 <part name="C4" library="Capacitors" deviceset="C0603C103K5RACTU" device="" package3d_urn="urn:adsk.eagle:package:24972866/1" value="10n/50V"/>
-<part name="U1" library="Nixie" deviceset="TM4C1231H6PMI7" device="" package3d_urn="urn:adsk.eagle:package:24923832/2"/>
+<part name="U1" library="ICs" deviceset="TM4C1231H6PMI7" device="" package3d_urn="urn:adsk.eagle:package:24923832/2"/>
 <part name="M1" library="Connectors" deviceset="JTAG-10PIN-ARM-CONN" device="" package3d_urn="urn:adsk.eagle:package:24925326/6"/>
 <part name="R1" library="Resistors" deviceset="CRCW0603100RFK" device="" package3d_urn="urn:adsk.eagle:package:24925614/1" value="100/1%"/>
@@
 <part name="R8" library="Resistors" deviceset="CRCW060333R0FK" device="" package3d_urn="urn:adsk.eagle:package:24925614/1" value="33/1%"/>
 <part name="R9" library="Resistors" deviceset="CRCW060333R0FK" device="" package3d_urn="urn:adsk.eagle:package:24925614/1" value="33/1%"/>
-<part name="Q1" library="Nixie" deviceset="NIXIE-IN-8-2" device=""/>
-<part name="Q2" library="Nixie" deviceset="NIXIE-IN-8-2" device=""/>
-<part name="Q3" library="Nixie" deviceset="NIXIE-IN-8-2" device=""/>
-<part name="Q4" library="Nixie" deviceset="NIXIE-IN-8-2" device=""/>
-<part name="IC9" library="Nixie" deviceset="SN75468" device="D" package3d_urn="urn:adsk.eagle:package:24873557/2"/>
-<part name="IC10" library="Nixie" deviceset="SN74HC595" device="PW" package3d_urn="urn:adsk.eagle:package:24918114/2"/>
+<part name="Q1" library="Misc" deviceset="NIXIE-IN-8-2" device=""/>
+<part name="Q2" library="Misc" deviceset="NIXIE-IN-8-2" device=""/>
+<part name="Q3" library="Misc" deviceset="NIXIE-IN-8-2" device=""/>
+<part name="Q4" library="Misc" deviceset="NIXIE-IN-8-2" device=""/>
+<part name="IC9" library="ICs" deviceset="SN75468" device="D" package3d_urn="urn:adsk.eagle:package:24873557/2"/>
+<part name="IC10" library="ICs" deviceset="SN74HC595" device="PW" package3d_urn="urn:adsk.eagle:package:24918114/2"/>
 <part name="C5" library="Capacitors" deviceset="C0603C103K5RACTU" device="" package3d_urn="urn:adsk.eagle:package:24972866/1" value="10n/50V"/>
 <part name="S1" library="Supplies" deviceset="3V3" device=""/>
@@
 <part name="S31" library="Supplies" deviceset="HV" device=""/>
 <part name="R14" library="Resistors" deviceset="CRCW060333R0FK" device="" package3d_urn="urn:adsk.eagle:package:24925614/1" value="33/1%"/>
+<part name="PS1" library="Misc" deviceset="S8421-45R" device="" package3d_urn="urn:adsk.eagle:package:24998728/2" value="S8421-45R"/>
+<part name="S32" library="Supplies" deviceset="GND" device=""/>
 </parts>
 <sheets>
@@
 <attribute name="VALUE" x="-137.16" y="-70.612" size="1.27" layer="96" align="bottom-center"/>
 </instance>
-<instance part="C6" gate="A" x="-205.74" y="17.78" smashed="yes">
-<attribute name="NAME" x="-203.2" y="18.796" size="1.27" layer="95"/>
-<attribute name="VALUE" x="-203.2" y="17.145" size="1.016" layer="96"/>
-<attribute name="PACKAGE" x="-203.2" y="15.748" size="1.016" layer="96"/>
-</instance>
-<instance part="S29" gate="G$1" x="-205.74" y="12.7" smashed="yes">
-<attribute name="VALUE" x="-205.74" y="8.128" size="1.27" layer="96" align="bottom-center"/>
+<instance part="C6" gate="A" x="-236.22" y="17.78" smashed="yes">
+<attribute name="NAME" x="-233.68" y="18.796" size="1.27" layer="95"/>
+<attribute name="VALUE" x="-233.68" y="17.145" size="1.016" layer="96"/>
+<attribute name="PACKAGE" x="-233.68" y="15.748" size="1.016" layer="96"/>
+</instance>
+<instance part="S29" gate="G$1" x="-236.22" y="12.7" smashed="yes">
+<attribute name="VALUE" x="-236.22" y="8.128" size="1.27" layer="96" align="bottom-center"/>
 </instance>
 <instance part="S30" gate="G$1" x="-205.74" y="53.34" smashed="yes">
@@
 <instance part="S31" gate="G$1" x="71.12" y="-137.16" smashed="yes">
 <attribute name="VALUE" x="71.12" y="-132.842" size="1.27" layer="96" align="bottom-center"/>
+</instance>
+<instance part="PS1" gate="A" x="-218.44" y="5.08" smashed="yes">
+<attribute name="NAME" x="-213.36" y="6.35" size="1.27" layer="95"/>
+<attribute name="VALUE" x="-213.36" y="3.81" size="1.27" layer="95"/>
+</instance>
+<instance part="S32" gate="G$1" x="-218.44" y="-5.08" smashed="yes">
+<attribute name="VALUE" x="-218.44" y="-9.652" size="1.27" layer="96" align="bottom-center"/>
 </instance>
 </instances>
@@
 <pinref part="S29" gate="G$1" pin="GND"/>
 <pinref part="C6" gate="A" pin="2"/>
-<wire x1="-205.74" y1="12.7" x2="-205.74" y2="15.24" width="0.1524" layer="91"/>
+<wire x1="-236.22" y1="12.7" x2="-236.22" y2="15.24" width="0.1524" layer="91"/>
+</segment>
+<segment>
+<pinref part="S32" gate="G$1" pin="GND"/>
+<pinref part="PS1" gate="A" pin="CATHODE"/>
+<wire x1="-218.44" y1="-5.08" x2="-218.44" y2="-2.54" width="0.1524" layer="91"/>
 </segment>
 </net>
@@
 <wire x1="-187.96" y1="22.86" x2="-185.42" y2="22.86" width="0.1524" layer="91"/>
 <pinref part="C6" gate="A" pin="1"/>
-<wire x1="-205.74" y1="22.86" x2="-187.96" y2="22.86" width="0.1524" layer="91"/>
-<wire x1="-205.74" y1="20.32" x2="-205.74" y2="22.86" width="0.1524" layer="91"/>
+<wire x1="-236.22" y1="22.86" x2="-187.96" y2="22.86" width="0.1524" layer="91"/>
+<wire x1="-236.22" y1="20.32" x2="-236.22" y2="22.86" width="0.1524" layer="91"/>
 <junction x="-187.96" y="22.86"/>
 </segment>
@@
 </segment>
 </net>
+<net name="VBAT" class="0">
+<segment>
+<pinref part="PS1" gate="A" pin="ANODE"/>
+<pinref part="U1" gate="A" pin="VBAT"/>
+<wire x1="-218.44" y1="12.7" x2="-218.44" y2="15.24" width="0.1524" layer="91"/>
+<wire x1="-218.44" y1="15.24" x2="-185.42" y2="15.24" width="0.1524" layer="91"/>
+</segment>
+</net>

Commit message: Update
Parts:
- removed R1: 100/1%, Resistors:CRCW0603100RFK
- removed R14, R6, R7, R8, R9: 33/1%, Resistors:CRCW060333R0FK
- removed R2: 10k/1%, Resistors:CRCW060310K0FK
- added C7: 10n/50V, Capacitors:C0603C103K5RACTU
- added C8: 1u/25V, Capacitors:CL10A105KA8NNNC
- added IC11: TPS73633DBVT, ICs:TPS73633DBVT
- added IC12: MCP111T-300E/TT, ICs:MCP111T-300E/TT
- added R15: 10k/1%, Resistors:CRCW060310K0FK
Connections:
- removed net N$39: M1.1/VCC, R1.P$1
- removed net N$40: M1.2/TMS, R6.P$1
- removed net N$41: M1.4/TCK, R7.P$1
- removed net N$42: M1.6/TDO, R8.P$1
- removed net N$43: M1.8/TDI, R9.P$1
- removed net N$56: M1.!10/RST, R14.P$1
- new net 12V: C8.1, IC11.EN, IC11.IN
- new net N$70: C7.1, IC11.NR
- net !JTAG_RST: now also IC12.OUT, M1.!10/RST, R15.P$1; no longer R14.P$2
- net 3V3: now also IC11.OUT, IC12.VDD, M1.1/VCC, R15.P$2; no longer R1.P$2
- net GND: now also C7.2, C8.2, IC11.GND, IC12.GND; no longer R2.P$1
- net JTAG_TCK: now also M1.4/TCK; no longer R7.P$2
- net JTAG_TDI: now also M1.8/TDI; no longer R9.P$2
- net JTAG_TDO: now also M1.6/TDO; no longer R2.P$2, R8.P$2
- net JTAG_TMS: now also M1.2/TMS; no longer R6.P$2

Commit message: Update
Parts:
- added C10, C9: 43p/50V, Capacitors:C0603C430J5GACTU
- added Y1: 16MHz, ICs:ABM8G-16.000MHZ-18-D2Y-T
Connections:
- new net N$39: C9.1, U1.OSC0, Y1.1
- new net N$40: C10.1, U1.OSC1, Y1.2
- net GND: now also C10.2, C9.2
Changed lines of the file:
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@@
 <part name="S36" library="Supplies" deviceset="3V3" device=""/>
 <part name="S37" library="Supplies" deviceset="3V3" device=""/>
+<part name="Y1" library="ICs" deviceset="ABM8G-16.000MHZ-18-D2Y-T" device="" package3d_urn="urn:adsk.eagle:package:25022963/1" value="16MHz"/>
+<part name="C9" library="Capacitors" deviceset="C0603C430J5GACTU" device="" package3d_urn="urn:adsk.eagle:package:25020390/1" value="43p/50V"/>
+<part name="C10" library="Capacitors" deviceset="C0603C430J5GACTU" device="" package3d_urn="urn:adsk.eagle:package:25020390/1" value="43p/50V"/>
+<part name="S38" library="Supplies" deviceset="GND" device=""/>
+<part name="S39" library="Supplies" deviceset="GND" device=""/>
 </parts>
 <sheets>
@@
 <attribute name="VALUE" x="25.4" y="-60.452" size="1.27" layer="96" align="bottom-center"/>
 </instance>
-<instance part="C6" gate="A" x="-45.72" y="27.94" smashed="yes">
-<attribute name="NAME" x="-43.18" y="28.956" size="1.27" layer="95"/>
-<attribute name="VALUE" x="-43.18" y="27.305" size="1.016" layer="96"/>
-<attribute name="PACKAGE" x="-43.18" y="25.908" size="1.016" layer="96"/>
-</instance>
-<instance part="S29" gate="A" x="-45.72" y="22.86" smashed="yes">
-<attribute name="VALUE" x="-45.72" y="18.288" size="1.27" layer="96" align="bottom-center"/>
+<instance part="C6" gate="A" x="-43.18" y="27.94" smashed="yes">
+<attribute name="NAME" x="-40.64" y="28.956" size="1.27" layer="95"/>
+<attribute name="VALUE" x="-40.64" y="27.305" size="1.016" layer="96"/>
+<attribute name="PACKAGE" x="-40.64" y="25.908" size="1.016" layer="96"/>
+</instance>
+<instance part="S29" gate="A" x="-43.18" y="22.86" smashed="yes">
+<attribute name="VALUE" x="-43.18" y="18.288" size="1.27" layer="96" align="bottom-center"/>
 </instance>
 <instance part="S30" gate="A" x="-50.8" y="60.96" smashed="yes">
 <attribute name="VALUE" x="-50.8" y="65.278" size="1.27" layer="96" align="bottom-center"/>
 </instance>
-<instance part="PS1" gate="A" x="-78.74" y="-45.72" smashed="yes" grouprefs="COIN_CELL_BATTERY_SOCKET">
-<attribute name="NAME" x="-73.66" y="-44.45" size="1.27" layer="95"/>
-<attribute name="VALUE" x="-73.66" y="-46.99" size="1.27" layer="95"/>
-</instance>
-<instance part="S32" gate="A" x="-78.74" y="-55.88" smashed="yes" grouprefs="COIN_CELL_BATTERY_SOCKET">
-<attribute name="VALUE" x="-78.74" y="-60.452" size="1.27" layer="96" align="bottom-center"/>
+<instance part="PS1" gate="A" x="-91.44" y="-43.18" smashed="yes" grouprefs="COIN_CELL_BATTERY_SOCKET">
+<attribute name="NAME" x="-86.36" y="-41.91" size="1.27" layer="95"/>
+<attribute name="VALUE" x="-86.36" y="-44.45" size="1.27" layer="95"/>
+</instance>
+<instance part="S32" gate="A" x="-91.44" y="-53.34" smashed="yes" grouprefs="COIN_CELL_BATTERY_SOCKET">
+<attribute name="VALUE" x="-91.44" y="-57.912" size="1.27" layer="96" align="bottom-center"/>
 </instance>
 <instance part="IC11" gate="A" x="-71.12" y="50.8" smashed="yes">
 <attribute name="NAME" x="-78.74" y="56.642" size="1.778" layer="95"/>
 <attribute name="VALUE" x="-78.74" y="43.18" size="1.778" layer="96"/>
+<attribute name="PACKAGE" x="-78.74" y="40.64" size="1.27" layer="96" ratio="6" rot="SR0"/>
 </instance>
 <instance part="C7" gate="A" x="-55.88" y="43.18" smashed="yes">
@@
 <attribute name="NAME" x="60.96" y="26.162" size="1.778" layer="95"/>
 <attribute name="VALUE" x="60.96" y="12.7" size="1.778" layer="96"/>
+<attribute name="PACKAGE" x="60.96" y="10.16" size="1.27" layer="96" ratio="6" rot="SR0"/>
 </instance>
 <instance part="M1" gate="A" x="73.66" y="-43.18" smashed="yes" grouprefs="JTAG_CONNECTOR">
@@
 <instance part="S37" gate="A" x="88.9" y="38.1" smashed="yes" grouprefs="RESET_SUPERVISOR">
 <attribute name="VALUE" x="88.9" y="42.418" size="1.27" layer="96" align="bottom-center"/>
+</instance>
+<instance part="Y1" gate="A" x="-48.26" y="0" smashed="yes">
+<attribute name="NAME" x="-50.8" y="3.302" size="1.778" layer="95"/>
+<attribute name="VALUE" x="-50.8" y="-4.318" size="1.27" layer="95"/>
+<attribute name="PACKAGE" x="-50.8" y="-6.35" size="1.27" layer="96" ratio="6" rot="SR0"/>
+</instance>
+<instance part="C9" gate="A" x="-60.96" y="-7.62" smashed="yes">
+<attribute name="NAME" x="-58.42" y="-6.604" size="1.27" layer="95"/>
+<attribute name="VALUE" x="-58.42" y="-8.255" size="1.016" layer="96"/>
+<attribute name="PACKAGE" x="-58.42" y="-9.652" size="1.016" layer="96"/>
+</instance>
+<instance part="C10" gate="A" x="-35.56" y="-7.62" smashed="yes">
+<attribute name="NAME" x="-33.02" y="-6.604" size="1.27" layer="95"/>
+<attribute name="VALUE" x="-33.02" y="-8.255" size="1.016" layer="96"/>
+<attribute name="PACKAGE" x="-33.02" y="-9.652" size="1.016" layer="96"/>
+</instance>
+<instance part="S38" gate="A" x="-60.96" y="-12.7" smashed="yes">
+<attribute name="VALUE" x="-60.96" y="-17.272" size="1.27" layer="96" align="bottom-center"/>
+</instance>
+<instance part="S39" gate="A" x="-35.56" y="-12.7" smashed="yes">
+<attribute name="VALUE" x="-35.56" y="-17.272" size="1.27" layer="96" align="bottom-center"/>
 </instance>
 </instances>
@@
 <pinref part="S29" gate="A" pin="GND"/>
 <pinref part="C6" gate="A" pin="2"/>
-<wire x1="-45.72" y1="22.86" x2="-45.72" y2="25.4" width="0.1524" layer="91"/>
+<wire x1="-43.18" y1="22.86" x2="-43.18" y2="25.4" width="0.1524" layer="91"/>
 </segment>
 <segment>
 <pinref part="S32" gate="A" pin="GND"/>
 <pinref part="PS1" gate="A" pin="CATHODE"/>
-<wire x1="-78.74" y1="-55.88" x2="-78.74" y2="-53.34" width="0.1524" layer="91" grouprefs="COIN_CELL_BATTERY_SOCKET"/>
+<wire x1="-91.44" y1="-53.34" x2="-91.44" y2="-50.8" width="0.1524" layer="91" grouprefs="COIN_CELL_BATTERY_SOCKET"/>
 </segment>
 <segment>
@@
 <wire x1="55.88" y1="17.78" x2="55.88" y2="12.7" width="0.1524" layer="91" grouprefs="RESET_SUPERVISOR"/>
 </segment>
+<segment>
+<pinref part="C9" gate="A" pin="2"/>
+<pinref part="S38" gate="A" pin="GND"/>
+<wire x1="-60.96" y1="-10.16" x2="-60.96" y2="-12.7" width="0.1524" layer="91"/>
+</segment>
+<segment>
+<pinref part="C10" gate="A" pin="2"/>
+<pinref part="S39" gate="A" pin="GND"/>
+<wire x1="-35.56" y1="-10.16" x2="-35.56" y2="-12.7" width="0.1524" layer="91"/>
+</segment>
 </net>
 <net name="U1_VDDC" class="0">
@@
 <wire x1="-25.4" y1="33.02" x2="-22.86" y2="33.02" width="0.1524" layer="91"/>
 <pinref part="C6" gate="A" pin="1"/>
-<wire x1="-45.72" y1="33.02" x2="-25.4" y2="33.02" width="0.1524" layer="91"/>
-<wire x1="-45.72" y1="30.48" x2="-45.72" y2="33.02" width="0.1524" layer="91"/>
+<wire x1="-43.18" y1="33.02" x2="-25.4" y2="33.02" width="0.1524" layer="91"/>
+<wire x1="-43.18" y1="30.48" x2="-43.18" y2="33.02" width="0.1524" layer="91"/>
 <junction x="-25.4" y="33.02"/>
 </segment>
@@
 <segment>
 <pinref part="PS1" gate="A" pin="ANODE"/>
-<wire x1="-78.74" y1="-38.1" x2="-78.74" y2="-35.56" width="0.1524" layer="91" grouprefs="COIN_CELL_BATTERY_SOCKET"/>
-<label x="-78.74" y="-34.798" size="1.27" layer="95" align="bottom-center" grouprefs="COIN_CELL_BATTERY_SOCKET"/>
+<wire x1="-91.44" y1="-35.56" x2="-91.44" y2="-33.02" width="0.1524" layer="91" grouprefs="COIN_CELL_BATTERY_SOCKET"/>
+<label x="-91.44" y="-32.258" size="1.27" layer="95" align="bottom-center" grouprefs="COIN_CELL_BATTERY_SOCKET"/>
 </segment>
 <segment>
@@
 </segment>
 </net>
+<net name="N$39" class="0">
+<segment>
+<pinref part="U1" gate="A" pin="OSC0"/>
+<pinref part="C9" gate="A" pin="1"/>
+<wire x1="-22.86" y1="10.16" x2="-60.96" y2="10.16" width="0.1524" layer="91"/>
+<wire x1="-60.96" y1="10.16" x2="-60.96" y2="0" width="0.1524" layer="91"/>
+<pinref part="Y1" gate="A" pin="1"/>
+<wire x1="-60.96" y1="0" x2="-60.96" y2="-5.08" width="0.1524" layer="91"/>
+<wire x1="-53.34" y1="0" x2="-60.96" y2="0" width="0.1524" layer="91"/>
+<junction x="-60.96" y="0"/>
+</segment>
+</net>
+<net name="N$40" class="0">
+<segment>
+<pinref part="C10" gate="A" pin="1"/>
+<pinref part="U1" gate="A" pin="OSC1"/>
+<wire x1="-35.56" y1="-5.08" x2="-35.56" y2="0" width="0.1524" layer="91"/>
+<wire x1="-35.56" y1="0" x2="-35.56" y2="5.08" width="0.1524" layer="91"/>
+<wire x1="-35.56" y1="5.08" x2="-22.86" y2="5.08" width="0.1524" layer="91"/>
+<pinref part="Y1" gate="A" pin="2"/>
+<wire x1="-43.18" y1="0" x2="-35.56" y2="0" width="0.1524" layer="91"/>
+<junction x="-35.56" y="0"/>
+</segment>
+</net>
 </nets>
 </sheet>
-<sheet>
-<description>JTAG_INTERFACE</description>
-<plain>
-</plain>
-<instances>
-</instances>
-<busses>
-</busses>
-<nets>
-</nets>
-</sheet>
