File: NixieClock.sch (EAGLE design)
At the start: 39 parts, among them IC1 SN75468D, IC10 SN74HC595PW, IC11 TPS73633DBVT, IC12 MCP111T-300E/TT, IC2 SN75468D, IC3 SN75468D, IC4 SN75468D, IC5 SN74HC595PW, IC6 SN74HC595PW, IC7 SN74HC595PW, IC8 SN74HC595PW, IC9 SN75468D, M1 JTAG-10PIN-ARM-CONN, Q1 NIXIE-IN-8-2, Q2 NIXIE-IN-8-2, Q3 NIXIE-IN-8-2, Q4 NIXIE-IN-8-2, U1 TM4C1231H6PMI7, Y1 16MHz

Commit message: Update
Parts:
- added C11, C12: 30p/50V, Capacitors:C0603C300J5GACTU
- added C13: 470u/16V, Capacitors:ECA1CM471
- added C14: 4u7/250V, Capacitors:ECA2EHG4R7
- added C15, C17: 100n/50V, Capacitors:C0603C104M5RACTU
- added C16: 10u/25V, Capacitors:C0603C103K5RACTU
- added D2: ES2G-E3/52T, Diodes:ES2G-E3/52T
- added D3: PMEG4030ER, Diodes:PMEG4010CEJ
- added IC13: MAX1771ESA+, ICs:MAX1771ESA+
- added J1, J2: PCB Terminal, Connectors:PCB_TERMINAL_2.8X0.81_RGIHT_ANGLE
- added J3: 501568-0607, Connectors:MOLEX_501568-0607
- added L1: MCSDRH125B-101MHF, Inductors:MCSDRH125B-101MHF
- added Q5: BF722, Transistors:BF722
- added Q6: BF723, Transistors:BF723
- added Q7: FQD16N25CTM, Transistors:FQD16N25CTM
- added R1: 1M/1%, Resistors:CRCW06031M00FKEA
- added R14, R8: 100k/1%, Resistors:CRCW0603100KFKEA
- added R16: 5k/10%, Resistors:T93YB502KT20
- added R2: 0.05/1%, Resistors:ERJ8CWFR050V
- added R6: 1.5M/1%, Resistors:MCPWR12FTEA1504
- added R7: 10k/1%, Resistors:CRCW060310K0FKEA
- added R9: 91k/1%, Resistors:ERJP06F9102V
- added Y2: 32.768 kHz, ICs:ABS25-32.768KHZ-1-T
- C1, C2, C3, C4, C5, C7: value 10n/50V -> 10u/25V
- R10, R11, R12, R13: device Resistors:CRCW121010K0FK -> Resistors:CRCW121010K0FKEA
- R15, R3, R4: device Resistors:CRCW060310K0FK -> Resistors:CRCW060310K0FKEA
- R5: device Resistors:CRCW06031M00FK -> Resistors:CRCW06031M00FKEA
- Y1: value 16MHz -> 16 MHz
Connections:
- net N$39 renamed OSC0
- net N$40 renamed OSC1
- new net !WAKE: R1.1, U1.!WAKE
- new net MCU_PWM: R14.1, U1.PB6
- new net N$39: J3.1, U1.PE0
- new net N$40: J3.2, U1.PE1
- new net N$41: J3.3, U1.PE2
- new net N$42: D3.2, J1.1
- new net N$43: J3.5, U1.PE4
- new net N$56: IC13.EXT, Q7.G
- new net N$71: IC13.CS, Q7.S, R2.2
- new net N$72: D2.2, L1.2, Q7.D
- new net N$73: C14.1, D2.1, Q6.E, R6.2, R8.1
- new net N$77: C15.1, IC13.REF
- new net N$78: Q6.B, R8.2, R9.2
- new net N$79: Q5.C, R9.1
- new net N$80: Q5.B, R14.2
- new net N$81: IC13.FB, R16.1, R6.1
- new net N$83: R16.2, R16.3, R7.2
- new net XOSC0: C12.1, U1.XOSC0, Y2.2
- new net XOSC1: C11.1, U1.XOSC1, Y2.1
- net !JTAG_RST: now also R15.1; no longer R15.P$1
- net 12V: now also C13.1, C16.1, C17.1, D3.1, IC13.V+, L1.1
- net 3V3: now also R1.2, R15.2, R3.2, R4.2; no longer R15.P$2, R3.P$2, R4.P$2
- net DTA_COM: now also R5.1; no longer R5.P$1
- net GND: now also C11.2, C12.2, C13.2, C14.2, C15.2, C16.2, C17.2, IC13.AGND, IC13.GND, IC13.SHDN, J2.1, J3.4, J3.6, Q5.E, R2.1, R7.1
- net HV: now also Q6.C, R10.2, R11.2, R12.2, R13.2, R5.2; no longer R10.P$2, R11.P$2, R12.P$2, R13.P$2, R5.P$2
- net JTAG_TCK: now also R4.1; no longer R4.P$1
- net JTAG_TMS: now also R3.1; no longer R3.P$1
- net N$55: now also R10.1; no longer R10.P$1
- net N$74: now also R11.1; no longer R11.P$1
- net N$75: now also R12.1; no longer R12.P$1
- net N$76: now also R13.1; no longer R13.P$1
Other:
- note added: "150V...220V"

Commit message: Update
Connections:
- net N$42 renamed VSUPP
- net N$73 renamed PRE_HV
Changed lines of the file:
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@@
 <class number="0" name="default" width="0" drill="0">
+</class>
+<class number="1" name="Supply" width="1" drill="0">
 </class>
 </classes>
@@
 <part name="S29" library="Supplies" deviceset="GND" device=""/>
 <part name="S30" library="Supplies" deviceset="3V3" device=""/>
-<part name="PS1" library="Misc" deviceset="S8421-45R" device="" package3d_urn="urn:adsk.eagle:package:24998728/2" value="S8421-45R"/>
+<part name="PS1" library="Misc" deviceset="S8421-45R" device="" package3d_urn="urn:adsk.eagle:package:24998728/4" value="S8421-45R"/>
 <part name="S32" library="Supplies" deviceset="GND" device=""/>
 <part name="IC11" library="ICs" deviceset="TPS73633DBVT" device="" package3d_urn="urn:adsk.eagle:package:25020238/2"/>
@@
 </segment>
 </net>
-<net name="N$42" class="0">
+<net name="VSUPP" class="1">
 <segment>
 <pinref part="J1" gate="A" pin="1"/>
@@
 </segment>
 </net>
-<net name="N$73" class="0">
+<net name="PRE_HV" class="0">
 <segment>
 <pinref part="D2" gate="A" pin="1"/>

Commit message: Update
Parts:
- Y2: device ICs:ABS25-32.768KHZ-1-T -> ICs:ABS07AIG-32.768KHZ-1-T
Changed lines of the file:
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@@
 <part name="S38" library="Supplies" deviceset="GND" device=""/>
 <part name="S39" library="Supplies" deviceset="GND" device=""/>
-<part name="Y2" library="ICs" deviceset="ABS25-32.768KHZ-1-T" device="" package3d_urn="urn:adsk.eagle:package:25030719/2" value="32.768 kHz"/>
+<part name="Y2" library="ICs" deviceset="ABS07AIG-32.768KHZ-1-T" device="" package3d_urn="urn:adsk.eagle:package:25206263/2" value="32.768 kHz"/>
 <part name="C11" library="Capacitors" deviceset="C0603C300J5GACTU" device="" package3d_urn="urn:adsk.eagle:package:25020390/1" value="30p/50V"/>
 <part name="C12" library="Capacitors" deviceset="C0603C300J5GACTU" device="" package3d_urn="urn:adsk.eagle:package:25020390/1" value="30p/50V"/>
