File: NixieClock.sch (EAGLE design)
At the start: 65 parts, among them IC1 SN75468D, IC10 SN74HC595PW, IC11 TPS73633DBVT, IC12 MCP111T-300E/TT, IC13 MAX1771ESA+, IC2 SN75468D, IC3 SN75468D, IC4 SN75468D, IC5 SN74HC595PW, IC6 SN74HC595PW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

Commit message: Update
Parts:
- C1, C16, C2, C3, C4, C5, C7: value 10u/25V -> 10n/50V
Changed lines of the file:
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@@
 <part name="IC7" library="ICs" deviceset="SN74HC595" device="PW" package3d_urn="urn:adsk.eagle:package:24918114/2"/>
 <part name="IC8" library="ICs" deviceset="SN74HC595" device="PW" package3d_urn="urn:adsk.eagle:package:24918114/2"/>
-<part name="C1" library="Capacitors" deviceset="C0603C103K5RACTU" device="" package3d_urn="urn:adsk.eagle:package:25131932/1" value="10u/25V"/>
-<part name="C2" library="Capacitors" deviceset="C0603C103K5RACTU" device="" package3d_urn="urn:adsk.eagle:package:25131932/1" value="10u/25V"/>
-<part name="C3" library="Capacitors" deviceset="C0603C103K5RACTU" device="" package3d_urn="urn:adsk.eagle:package:25131932/1" value="10u/25V"/>
-<part name="C4" library="Capacitors" deviceset="C0603C103K5RACTU" device="" package3d_urn="urn:adsk.eagle:package:25131932/1" value="10u/25V"/>
+<part name="C1" library="Capacitors" deviceset="C0603C103K5RACTU" device="" package3d_urn="urn:adsk.eagle:package:25020390/1" value="10n/50V"/>
+<part name="C2" library="Capacitors" deviceset="C0603C103K5RACTU" device="" package3d_urn="urn:adsk.eagle:package:25020390/1" value="10n/50V"/>
+<part name="C3" library="Capacitors" deviceset="C0603C103K5RACTU" device="" package3d_urn="urn:adsk.eagle:package:25020390/1" value="10n/50V"/>
+<part name="C4" library="Capacitors" deviceset="C0603C103K5RACTU" device="" package3d_urn="urn:adsk.eagle:package:25020390/1" value="10n/50V"/>
 <part name="Q1" library="Misc" deviceset="NIXIE-IN-8-2" device=""/>
 <part name="Q2" library="Misc" deviceset="NIXIE-IN-8-2" device=""/>
@@
 <part name="IC9" library="ICs" deviceset="SN75468" device="D" package3d_urn="urn:adsk.eagle:package:24873557/2"/>
 <part name="IC10" library="ICs" deviceset="SN74HC595" device="PW" package3d_urn="urn:adsk.eagle:package:24918114/2"/>
-<part name="C5" library="Capacitors" deviceset="C0603C103K5RACTU" device="" package3d_urn="urn:adsk.eagle:package:25131932/1" value="10u/25V"/>
+<part name="C5" library="Capacitors" deviceset="C0603C103K5RACTU" device="" package3d_urn="urn:adsk.eagle:package:25020390/1" value="10n/50V"/>
 <part name="S1" library="Supplies" deviceset="3V3" device=""/>
 <part name="S2" library="Supplies" deviceset="3V3" device=""/>
@@
 <part name="S32" library="Supplies" deviceset="GND" device=""/>
 <part name="IC11" library="ICs" deviceset="TPS73633DBVT" device="" package3d_urn="urn:adsk.eagle:package:25020238/2"/>
-<part name="C7" library="Capacitors" deviceset="C0603C103K5RACTU" device="" package3d_urn="urn:adsk.eagle:package:25131932/1" value="10u/25V"/>
+<part name="C7" library="Capacitors" deviceset="C0603C103K5RACTU" device="" package3d_urn="urn:adsk.eagle:package:25020390/1" value="10n/50V"/>
 <part name="C8" library="Capacitors" deviceset="CL10A105KA8NNNC" device="" package3d_urn="urn:adsk.eagle:package:25020390/1" value="1u/25V"/>
 <part name="S33" library="Supplies" deviceset="12V" device=""/>
@@
 <part name="S52" library="Supplies" deviceset="GND" device=""/>
 <part name="S53" library="Supplies" deviceset="GND" device=""/>
-<part name="C16" library="Capacitors" deviceset="C0603C103K5RACTU" device="" package3d_urn="urn:adsk.eagle:package:25131932/1" value="10u/25V"/>
+<part name="C16" library="Capacitors" deviceset="C0603C103K5RACTU" device="" package3d_urn="urn:adsk.eagle:package:25020390/1" value="10n/50V"/>
 <part name="C17" library="Capacitors" deviceset="C0603C104M5RACTU" device="" package3d_urn="urn:adsk.eagle:package:25020390/1" value="100n/50V"/>
 <part name="S54" library="Supplies" deviceset="GND" device=""/>

Commit message: Update
Parts:
- removed C5: 10n/50V, Capacitors:C0603C103K5RACTU
- removed IC10: SN74HC595PW, ICs:SN74HC595PW
- removed IC9: SN75468D, ICs:SN75468D
- added Q8: BF820, Transistors:BF820
- added R17, R18: 100k/1%, Resistors:CRCW0603100KFKEA
- C16: value 10n/50V -> 10u/25V; device Capacitors:C0603C103K5RACTU -> Capacitors:C1206C106K3PACTU
- Q5: value BF722 -> BF820; device Transistors:BF722 -> Transistors:BF820
- Q6: value BF723 -> BF821; device Transistors:BF723 -> Transistors:BF821
Connections:
- net U1_VDDC renamed MCU_VDDC
- removed net N$27 (its old number): IC4.3B, IC8.QC
- removed net N$34 (its old number): IC1.3C, Q1.K2
- removed net N$47 (its old number): IC2.3C, Q2.K6
- removed net N$69: IC4.7C, Q4.K8
- new net N$12: IC1.4C, Q2.K1
- new net N$20: IC2.4C, Q2.K8
- new net N$28: IC2.3B, IC6.QE
- new net N$42: IC4.6C, Q4.K4
- net 3V3: no longer C5.1, IC10.!SRCLR, IC10.VCC
- net DTA_COM: no longer IC9.COM
- net GND: now also Q8.E, R17.2; no longer C5.2, IC10.!OE, IC10.GND, IC9.2B, IC9.3B, IC9.4B, IC9.5B, IC9.6B, IC9.7B, IC9.E
- net N$1: now also IC1.7B; no longer IC1.1B
- net N$10: now also IC1.6C, Q1.K2; no longer IC2.2B, IC6.QB
- net N$11: now also IC1.5C, Q1.K0; no longer IC2.3B, IC6.QC
- net N$13: now also IC1.3C, Q2.K2; no longer IC2.5B, IC6.QE
- net N$14: now also IC1.2C, Q2.K3; no longer IC2.6B, IC6.QF
- net N$15: now also IC1.1C, Q2.K4; no longer IC2.7B, IC6.QG
- net N$17: now also IC2.7C, Q2.K5; no longer IC3.1B, IC7.QA
- net N$18: now also IC2.6C, Q2.K6; no longer IC3.2B, IC7.QB
- net N$19: now also IC2.5C, Q2.K7; no longer IC3.3B, IC7.QC
- net N$2: now also IC1.6B; no longer IC1.2B
- net N$21: now also IC2.3C, Q2.K9; no longer IC3.5B, IC7.QE
- net N$22: now also IC2.2C, Q2.K0; no longer IC3.6B, IC7.QF
- net N$23: now also IC2.7B, IC6.QA; no longer IC3.7B, IC7.QG
- net N$25: now also IC2.6B, IC6.QB; no longer IC4.1B, IC8.QA
- net N$26: now also IC2.5B, IC6.QC; no longer IC4.2B, IC8.QB
- net N$29: now also IC2.2B, IC6.QF; no longer IC4.5B, IC8.QE
- net N$3: now also IC1.5B; no longer IC1.3B
- net N$30: now also IC2.1B, IC6.QG; no longer IC4.6B, IC8.QF
- net N$31: now also IC3.7B, IC7.QA; no longer IC4.7B, IC8.QG
- net N$32: now also IC3.6B, IC7.QB; no longer IC1.1C, Q1.K0
- net N$33: now also IC3.5B, IC7.QC; no longer IC1.2C, Q1.K1
- net N$35: now also IC3.3B, IC7.QE; no longer IC1.4C, Q2.K0
- net N$36: now also IC3.2B, IC7.QF; no longer IC1.5C, Q2.K1
- net N$37: now also IC3.1B, IC7.QG; no longer IC1.6C, Q2.K2
- net N$38: now also IC8.QH, R18.1; no longer IC9.1C, Q4.K9
- net N$44: now also IC4.7B, IC8.QA; no longer IC1.7C, Q2.K3
- net N$45: now also IC4.6B, IC8.QB; no longer IC2.1C, Q2.K4
- net N$46: now also IC4.5B, IC8.QC; no longer IC2.2C, Q2.K5
- net N$48: now also IC4.3B, IC8.QE; no longer IC2.4C, Q2.K7
- net N$49: now also IC4.2B, IC8.QF; no longer IC2.5C, Q2.K8
- net N$5: now also IC1.3B; no longer IC1.5B
- net N$50: now also IC4.1B, IC8.QG; no longer IC2.6C, Q2.K9
- net N$51: now also IC2.1C, Q3.K1; no longer IC2.7C, Q3.K0
- net N$52: now also IC3.7C, Q3.K2; no longer IC3.1C, Q3.K1
- net N$53: now also IC3.6C, Q3.K3; no longer IC3.2C, Q3.K2
- net N$54: now also IC3.5C, Q3.K4; no longer IC3.3C, Q3.K3
- net N$57: now also Q3.K5; no longer Q3.K4
- net N$58: now also IC3.3C, Q3.K0; no longer IC3.5C, Q3.K5
- net N$59: now also IC3.2C, Q4.K1; no longer IC3.6C, Q4.K0
- net N$6: now also IC1.2B; no longer IC1.6B
- net N$60: now also IC3.1C, Q4.K2; no longer IC3.7C, Q4.K1
- net N$61: now also IC4.7C, Q4.K3; no longer IC4.1C, Q4.K2
- net N$62: now also IC4.5C, Q4.K5; no longer IC4.2C, Q4.K3
- net N$63: now also IC4.4C, Q4.K6; no longer IC4.3C, Q4.K4
- net N$64: now also IC4.3C, Q4.K7; no longer IC4.4C, Q4.K5
- net N$65: now also Q8.B, R17.1, R18.2; no longer IC10.SER, IC8.QH'
- net N$66: now also IC4.2C, Q4.K8; no longer IC10.QA, IC9.1B
- net N$67: now also IC4.1C, Q4.K9; no longer IC4.5C, Q4.K6
- net N$68: now also Q4.K0, Q8.C; no longer IC4.6C, Q4.K7
- net N$7: now also IC1.1B; no longer IC1.7B
- net N$9: now also IC1.7C, Q1.K1; no longer IC2.1B, IC6.QA
- net SR_RCLK: no longer IC10.RCLK
- net SR_SRCLK: no longer IC10.SRCLK
Other:
- moved on the sheet: Q3, Q4, R12, R13

Commit message: Update
Parts:
- added MT1, MT2, MT3, MT4: MOUNTING_HOLE_3MM, Misc:MOUNTING_HOLE_3MM
- J1, J2: device Connectors:PCB_TERMINAL_2.8X0.81_RGIHT_ANGLE -> Connectors:PCB_TERMINAL_PAD
Connections:
- net N$39 renamed SW_3
- net N$40 renamed SW_2
- net N$41 renamed SW_1
- net N$43 renamed LIGHT_SEN
- net GND: now also MT1.GND, MT2.GND, MT3.GND, MT4.GND
Changed lines of the file:
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@@
 <part name="S29" library="Supplies" deviceset="GND" device=""/>
 <part name="S30" library="Supplies" deviceset="3V3" device=""/>
-<part name="PS1" library="Misc" deviceset="S8421-45R" device="" package3d_urn="urn:adsk.eagle:package:24998728/4" value="S8421-45R"/>
+<part name="PS1" library="Misc" deviceset="S8421-45R" device="" package3d_urn="urn:adsk.eagle:package:24998728/5" value="S8421-45R"/>
 <part name="S32" library="Supplies" deviceset="GND" device=""/>
 <part name="IC11" library="ICs" deviceset="TPS73633DBVT" device="" package3d_urn="urn:adsk.eagle:package:25020238/2"/>
@@
 <part name="J3" library="Connectors" deviceset="MOLEX_501568-0607" device="" package3d_urn="urn:adsk.eagle:package:25035327/3" value="501568-0607"/>
 <part name="S43" library="Supplies" deviceset="GND" device=""/>
-<part name="J1" library="Connectors" deviceset="PCB_TERMINAL_2.8X0.81_RGIHT_ANGLE" device="" package3d_urn="urn:adsk.eagle:package:25040458/2" value="PCB Terminal"/>
-<part name="J2" library="Connectors" deviceset="PCB_TERMINAL_2.8X0.81_RGIHT_ANGLE" device="" package3d_urn="urn:adsk.eagle:package:25040458/2" value="PCB Terminal"/>
+<part name="J1" library="Connectors" deviceset="PCB_TERMINAL_PAD" device="" value="PCB Terminal"/>
+<part name="J2" library="Connectors" deviceset="PCB_TERMINAL_PAD" device="" value="PCB Terminal"/>
 <part name="FRAME1" library="frames" library_urn="urn:adsk.eagle:library:229" deviceset="A3L-LOC" device="" value="Nixie Control And Driver"/>
 <part name="FRAME2" library="frames" library_urn="urn:adsk.eagle:library:229" deviceset="A3L-LOC" device="" value="MCU And Connectors"/>
@@
 <part name="S10" library="Supplies" deviceset="GND" device=""/>
 <part name="R18" library="Resistors" deviceset="CRCW0603100KFKEA" device="" package3d_urn="urn:adsk.eagle:package:24925614/1" value="100k/1%"/>
+<part name="MT1" library="Misc" deviceset="MOUNTING_HOLE_3MM" device=""/>
+<part name="MT2" library="Misc" deviceset="MOUNTING_HOLE_3MM" device=""/>
+<part name="MT3" library="Misc" deviceset="MOUNTING_HOLE_3MM" device=""/>
+<part name="MT4" library="Misc" deviceset="MOUNTING_HOLE_3MM" device=""/>
+<part name="S5" library="Supplies" deviceset="GND" device=""/>
+<part name="S15" library="Supplies" deviceset="GND" device=""/>
+<part name="S20" library="Supplies" deviceset="GND" device=""/>
+<part name="S62" library="Supplies" deviceset="GND" device=""/>
 </parts>
 <sheets>
@@
 </segment>
 </net>
-<net name="N$39" class="0">
+<net name="SW_3" class="0">
 <segment>
 <pinref part="U1" gate="A" pin="PE0"/>
@@
 </segment>
 </net>
-<net name="N$40" class="0">
+<net name="SW_2" class="0">
 <segment>
 <pinref part="U1" gate="A" pin="PE1"/>
@@
 </segment>
 </net>
-<net name="N$41" class="0">
+<net name="SW_1" class="0">
 <segment>
 <pinref part="U1" gate="A" pin="PE2"/>
@@
 </segment>
 </net>
-<net name="N$43" class="0">
+<net name="LIGHT_SEN" class="0">
 <segment>
 <pinref part="U1" gate="A" pin="PE4"/>
@@
 </segment>
 </net>
+</nets>
+</sheet>
+<sheet>
+<description>Miscellaneous</description>
+<plain>
+</plain>
+<instances>
+<instance part="MT1" gate="A" x="-15.24" y="5.08" smashed="yes"/>
+<instance part="MT2" gate="A" x="-5.08" y="5.08" smashed="yes"/>
+<instance part="MT3" gate="A" x="5.08" y="5.08" smashed="yes"/>
+<instance part="MT4" gate="A" x="15.24" y="5.08" smashed="yes"/>
+<instance part="S5" gate="A" x="-15.24" y="-2.54" smashed="yes">
+<attribute name="VALUE" x="-15.24" y="-7.112" size="1.27" layer="96" align="bottom-center"/>
+</instance>
+<instance part="S15" gate="A" x="-5.08" y="-2.54" smashed="yes">
+<attribute name="VALUE" x="-5.08" y="-7.112" size="1.27" layer="96" align="bottom-center"/>
+</instance>
+<instance part="S20" gate="A" x="5.08" y="-2.54" smashed="yes">
+<attribute name="VALUE" x="5.08" y="-7.112" size="1.27" layer="96" align="bottom-center"/>
+</instance>
+<instance part="S62" gate="A" x="15.24" y="-2.54" smashed="yes">
+<attribute name="VALUE" x="15.24" y="-7.112" size="1.27" layer="96" align="bottom-center"/>
+</instance>
+</instances>
+<busses>
+</busses>
+<nets>
+<net name="GND" class="0">
+<segment>
+<pinref part="MT1" gate="A" pin="GND"/>
+<pinref part="S5" gate="A" pin="GND"/>
+<wire x1="-15.24" y1="2.54" x2="-15.24" y2="-2.54" width="0.1524" layer="91"/>
+</segment>
+<segment>
+<pinref part="MT2" gate="A" pin="GND"/>
+<pinref part="S15" gate="A" pin="GND"/>
+<wire x1="-5.08" y1="2.54" x2="-5.08" y2="-2.54" width="0.1524" layer="91"/>
+</segment>
+<segment>
+<pinref part="MT3" gate="A" pin="GND"/>
+<pinref part="S20" gate="A" pin="GND"/>
+<wire x1="5.08" y1="2.54" x2="5.08" y2="-2.54" width="0.1524" layer="91"/>
+</segment>
+<segment>
+<pinref part="MT4" gate="A" pin="GND"/>
+<pinref part="S62" gate="A" pin="GND"/>
+<wire x1="15.24" y1="2.54" x2="15.24" y2="-2.54" width="0.1524" layer="91"/>
+</segment>
+</net>

Commit message: Update
Parts:
- IC5, IC6, IC7, IC8: value SN74HC595PW -> SN74HC595DR; device ICs:SN74HC595PW -> ICs:SN74HC595DR
- M1: value JTAG-10PIN-ARM-CONN -> JTAG-ARM-10PIN-PLACEHOLDER; device Connectors:JTAG-10PIN-ARM-CONN -> Connectors:JTAG-ARM-10PIN-PLACEHOLDER
Changed lines of the file:
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@@
 <part name="IC3" library="ICs" deviceset="SN75468" device="D" package3d_urn="urn:adsk.eagle:package:24873557/2"/>
 <part name="IC4" library="ICs" deviceset="SN75468" device="D" package3d_urn="urn:adsk.eagle:package:24873557/2"/>
-<part name="IC5" library="ICs" deviceset="SN74HC595" device="PW" package3d_urn="urn:adsk.eagle:package:24918114/2"/>
-<part name="IC6" library="ICs" deviceset="SN74HC595" device="PW" package3d_urn="urn:adsk.eagle:package:24918114/2"/>
-<part name="IC7" library="ICs" deviceset="SN74HC595" device="PW" package3d_urn="urn:adsk.eagle:package:24918114/2"/>
-<part name="IC8" library="ICs" deviceset="SN74HC595" device="PW" package3d_urn="urn:adsk.eagle:package:24918114/2"/>
+<part name="IC5" library="ICs" deviceset="SN74HC595DR" device="" package3d_urn="urn:adsk.eagle:package:24873557/2"/>
+<part name="IC6" library="ICs" deviceset="SN74HC595DR" device="" package3d_urn="urn:adsk.eagle:package:24873557/2"/>
+<part name="IC7" library="ICs" deviceset="SN74HC595DR" device="" package3d_urn="urn:adsk.eagle:package:24873557/2"/>
+<part name="IC8" library="ICs" deviceset="SN74HC595DR" device="" package3d_urn="urn:adsk.eagle:package:24873557/2"/>
 <part name="C1" library="Capacitors" deviceset="C0603C103K5RACTU" device="" package3d_urn="urn:adsk.eagle:package:25020390/1" value="10n/50V"/>
 <part name="C2" library="Capacitors" deviceset="C0603C103K5RACTU" device="" package3d_urn="urn:adsk.eagle:package:25020390/1" value="10n/50V"/>
@@
 <part name="S34" library="Supplies" deviceset="GND" device=""/>
 <part name="IC12" library="ICs" deviceset="MCP111T-300E/TT" device="" package3d_urn="urn:adsk.eagle:package:25020091/3"/>
-<part name="M1" library="Connectors" deviceset="JTAG-10PIN-ARM-CONN" device="" package3d_urn="urn:adsk.eagle:package:24925326/6"/>
+<part name="M1" library="Connectors" deviceset="JTAG-ARM-10PIN-PLACEHOLDER" device="" package3d_urn="urn:adsk.eagle:package:25317759/2"/>
 <part name="R3" library="Resistors" deviceset="CRCW060310K0FKEA" device="" package3d_urn="urn:adsk.eagle:package:24925614/1" value="10k/1%"/>
 <part name="R4" library="Resistors" deviceset="CRCW060310K0FKEA" device="" package3d_urn="urn:adsk.eagle:package:24925614/1" value="10k/1%"/>
@@
 <part name="S10" library="Supplies" deviceset="GND" device=""/>
 <part name="R18" library="Resistors" deviceset="CRCW0603100KFKEA" device="" package3d_urn="urn:adsk.eagle:package:24925614/1" value="100k/1%"/>
-<part name="MT1" library="Misc" deviceset="MOUNTING_HOLE_3MM" device=""/>
-<part name="MT2" library="Misc" deviceset="MOUNTING_HOLE_3MM" device=""/>
-<part name="MT3" library="Misc" deviceset="MOUNTING_HOLE_3MM" device=""/>
-<part name="MT4" library="Misc" deviceset="MOUNTING_HOLE_3MM" device=""/>
+<part name="MT1" library="Misc" deviceset="MOUNTING_HOLE_3MM" device="" package3d_urn="urn:adsk.eagle:package:25316982/2"/>
+<part name="MT2" library="Misc" deviceset="MOUNTING_HOLE_3MM" device="" package3d_urn="urn:adsk.eagle:package:25316982/2"/>
+<part name="MT3" library="Misc" deviceset="MOUNTING_HOLE_3MM" device="" package3d_urn="urn:adsk.eagle:package:25316982/2"/>
+<part name="MT4" library="Misc" deviceset="MOUNTING_HOLE_3MM" device="" package3d_urn="urn:adsk.eagle:package:25316982/2"/>
 <part name="S5" library="Supplies" deviceset="GND" device=""/>
 <part name="S15" library="Supplies" deviceset="GND" device=""/>

Commit message: Update
Parts:
- added C18, C5: 100n/50V, Capacitors:C0603C104M5RACTU
- added IC10, IC9: TLC5973, ICs:TLC5973
- added LED1, LED2, LED3, LED4: CLX6E-FKC, Diodes:CLX6E-FKC
- added R19, R20: 3k3/1%, Resistors:MCWR06X3301FTL
Connections:
- new net LED_SDI: IC9.SDI, U1.PA1_U0TX
- new net N$39: IC9.OUT0, LED1.CRED
- new net N$40: IC9.OUT2, LED1.CBLUE
- new net N$41: IC9.OUT1, LED1.CGREEN
- new net N$43: IC10.OUT0, LED3.CRED
- new net N$69: IC10.OUT1, LED3.CGREEN
- new net N$73: IC10.OUT2, LED3.CBLUE
- new net N$82: LED3.ARED, LED4.CRED
- new net N$84: LED3.AGREEN, LED4.CGREEN
- new net N$85: LED3.ABLUE, LED4.CBLUE
- new net N$86: LED1.ARED, LED2.CRED
- new net N$87: LED1.AGREEN, LED2.CGREEN
- new net N$88: LED1.ABLUE, LED2.CBLUE
- new net N$90: IC9.IREF, R20.2
- new net N$91: IC10.IREF, R19.2
- new net N$93: IC10.SDI, IC9.SDO
- net 12V: now also LED2.ABLUE, LED2.AGREEN, LED2.ARED, LED4.ABLUE, LED4.AGREEN, LED4.ARED
- net 3V3: now also C18.1, C5.1, IC10.VCC, IC9.VCC
- net GND: now also C18.2, C5.2, IC10.GND, IC9.GND, R19.1, R20.1
- net N$51: now also Q3.K0; no longer Q3.K1
- net N$52: now also IC3.3C, Q3.K5; no longer IC3.7C, Q3.K2
- net N$53: now also IC3.4C, Q3.K4; no longer IC3.6C, Q3.K3
- net N$54: now also Q3.K3; no longer Q3.K4
- net N$57: now also IC3.6C, Q3.K2; no longer IC3.4C, Q3.K5
- net N$58: now also IC3.7C, Q3.K1; no longer IC3.3C, Q3.K0
Other:
- moved on the sheet: C1, C10, C11, C12, C2, C3, C4, C9, D1, IC1, IC2, IC3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

Commit message: Update
Parts:
- C10, C9: value 43p/50V -> 30p/50V; device Capacitors:C0603C430J5GACTU -> Capacitors:C0603C300J5GACTU
- C11, C12: value 30p/50V -> 20p/50V; device Capacitors:C0603C300J5GACTU -> Capacitors:C0603C200J1GACTU
Changed lines of the file:
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@@
 <part name="C3" library="Capacitors" deviceset="C0603C103K5RACTU" device="" package3d_urn="urn:adsk.eagle:package:25020390/1" value="10n/50V"/>
 <part name="C4" library="Capacitors" deviceset="C0603C103K5RACTU" device="" package3d_urn="urn:adsk.eagle:package:25020390/1" value="10n/50V"/>
-<part name="Q1" library="Misc" deviceset="NIXIE-IN-8-2" device=""/>
-<part name="Q2" library="Misc" deviceset="NIXIE-IN-8-2" device=""/>
-<part name="Q3" library="Misc" deviceset="NIXIE-IN-8-2" device=""/>
-<part name="Q4" library="Misc" deviceset="NIXIE-IN-8-2" device=""/>
+<part name="Q1" library="Misc" deviceset="NIXIE-IN-8-2" device="" package3d_urn="urn:adsk.eagle:package:25351611/2"/>
+<part name="Q2" library="Misc" deviceset="NIXIE-IN-8-2" device="" package3d_urn="urn:adsk.eagle:package:25351611/2"/>
+<part name="Q3" library="Misc" deviceset="NIXIE-IN-8-2" device="" package3d_urn="urn:adsk.eagle:package:25351611/2"/>
+<part name="Q4" library="Misc" deviceset="NIXIE-IN-8-2" device="" package3d_urn="urn:adsk.eagle:package:25351611/2"/>
 <part name="S1" library="Supplies" deviceset="3V3" device=""/>
 <part name="S2" library="Supplies" deviceset="3V3" device=""/>
@@
 <part name="S37" library="Supplies" deviceset="3V3" device=""/>
 <part name="Y1" library="ICs" deviceset="ABM8G-16.000MHZ-18-D2Y-T" device="" package3d_urn="urn:adsk.eagle:package:25022963/1" value="16 MHz"/>
-<part name="C9" library="Capacitors" deviceset="C0603C430J5GACTU" device="" package3d_urn="urn:adsk.eagle:package:25020390/1" value="43p/50V"/>
-<part name="C10" library="Capacitors" deviceset="C0603C430J5GACTU" device="" package3d_urn="urn:adsk.eagle:package:25020390/1" value="43p/50V"/>
+<part name="C9" library="Capacitors" deviceset="C0603C300J5GACTU" device="" package3d_urn="urn:adsk.eagle:package:25020390/1" value="30p/50V"/>
+<part name="C10" library="Capacitors" deviceset="C0603C300J5GACTU" device="" package3d_urn="urn:adsk.eagle:package:25020390/1" value="30p/50V"/>
 <part name="S38" library="Supplies" deviceset="GND" device=""/>
 <part name="S39" library="Supplies" deviceset="GND" device=""/>
 <part name="Y2" library="ICs" deviceset="ABS07AIG-32.768KHZ-1-T" device="" package3d_urn="urn:adsk.eagle:package:25206263/2" value="32.768 kHz"/>
-<part name="C11" library="Capacitors" deviceset="C0603C300J5GACTU" device="" package3d_urn="urn:adsk.eagle:package:25020390/1" value="30p/50V"/>
-<part name="C12" library="Capacitors" deviceset="C0603C300J5GACTU" device="" package3d_urn="urn:adsk.eagle:package:25020390/1" value="30p/50V"/>
+<part name="C11" library="Capacitors" deviceset="C0603C200J1GACTU" device="" package3d_urn="urn:adsk.eagle:package:25020390/1" value="20p/50V"/>
+<part name="C12" library="Capacitors" deviceset="C0603C200J1GACTU" device="" package3d_urn="urn:adsk.eagle:package:25020390/1" value="20p/50V"/>
 <part name="S40" library="Supplies" deviceset="GND" device=""/>
 <part name="S41" library="Supplies" deviceset="GND" device=""/>
