File: NixieClock.sch (EAGLE design)
At the start: 79 parts, among them IC1 SN75468D, IC10 TLC5973, IC11 TPS73633DBVT, IC12 MCP111T-300E/TT, IC13 MAX1771ESA+, IC2 SN75468D, IC3 SN75468D, IC4 SN75468D, IC5 SN74HC595DR, IC6 SN74HC595DR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

Commit message: Update
Parts:
- removed U1: TM4C1231H6PMI7, ICs:TM4C1231H6PMI7
- added C19, C21: 10n/50V, Capacitors:C0603C103K5RACTU
- added C20, C22: 100n/50V, Capacitors:C0603C104M5RACTU
- added IC14: TM4C1231H6PMI, ICs:TM4C1231H6PMI
- IC1, IC2, IC3, IC4: value SN75468D -> SN75468; device ICs:SN75468D -> ICs:SN75468
- R2: value 0.05/1% -> 0R05/1%
Connections:
- net !JTAG_RST: now also IC14.!RST; no longer U1.!RST
- net !WAKE: now also IC14.!WAKE; no longer U1.!WAKE
- net 3V3: now also C19.1, C20.1, C21.1, C22.1, IC14.VDD, IC14.VDDA, IC14.VDD_2, IC14.VDD_3, IC14.VDD_4; no longer U1.VDD, U1.VDDA, U1.VDD_2, U1.VDD_3, U1.VDD_4
- net GND: now also C19.2, C20.2, C21.2, C22.2, IC14.GND, IC14.GNDA, IC14.GNDX, IC14.GND_2, IC14.GND_3, IC14.GND_4; no longer U1.GND, U1.GNDA, U1.GNDX, U1.GND_2, U1.GND_3, U1.GND_4
- net JTAG_TCK: now also IC14.PC0_TCK_SWCLK; no longer U1.PC0_TCK_SWCLK
- net JTAG_TDI: now also IC14.PC2_TDI; no longer U1.PC2_TDI
- net JTAG_TDO: now also IC14.PC3_TDO_SWO; no longer U1.PC3_TDO_SWO
- net JTAG_TMS: now also IC14.PC1_TMS_SWDIO; no longer U1.PC1_TMS_SWDIO
- net LED_SDI: now also IC14.PA1_U0TX; no longer U1.PA1_U0TX
- net LIGHT_SEN: now also IC14.PE4; no longer U1.PE4
- net MCU_PWM: now also IC14.PB6; no longer U1.PB6
- net MCU_VDDC: now also IC14.VDDC, IC14.VDDC_2; no longer U1.VDDC, U1.VDDC_2
- net OSC0: now also IC14.OSC0; no longer U1.OSC0
- net OSC1: now also IC14.OSC1; no longer U1.OSC1
- net SR_RCLK: now also IC14.PD1; no longer U1.PD1
- net SR_SER: now also IC14.PD0; no longer U1.PD0
- net SR_SRCLK: now also IC14.PD2; no longer U1.PD2
- net SW_1: now also IC14.PE2; no longer U1.PE2
- net SW_2: now also IC14.PE1; no longer U1.PE1
- net SW_3: now also IC14.PE0; no longer U1.PE0
- net VBAT: now also IC14.VBAT; no longer U1.VBAT
- net XOSC0: now also IC14.XOSC0; no longer U1.XOSC0
- net XOSC1: now also IC14.XOSC1; no longer U1.XOSC1
Other:
- moved on the sheet: C10, C11, C12, C6, C9, J3, R1, Y1, Y2

Commit message: Update
Parts:
- added R21: 2k/1%, Resistors:CRCW06032K00FKEA
- C10, C9: value 30p/50V -> 12p/50V; device Capacitors:C0603C300J5GACTU -> Capacitors:C0603C120J5GACTU
- Y1: device ICs:ABM8G-16.000MHZ-18-D2Y-T -> Crystals:MCSJK-7U-16.00-10-10-80-B-10
- Y2: device ICs:ABS07AIG-32.768KHZ-1-T -> Crystals:ABS07AIG-32.768KHZ-1-T
Connections:
- new net N$89: IC14.OSC1, R21.2
- net OSC1: now also R21.1; no longer IC14.OSC1
Changed lines of the file:
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@@
 <part name="S36" library="Supplies" deviceset="3V3" device=""/>
 <part name="S37" library="Supplies" deviceset="3V3" device=""/>
-<part name="Y1" library="ICs" deviceset="ABM8G-16.000MHZ-18-D2Y-T" device="" package3d_urn="urn:adsk.eagle:package:25022963/1" value="16 MHz"/>
-<part name="C9" library="Capacitors" deviceset="C0603C300J5GACTU" device="" package3d_urn="urn:adsk.eagle:package:25020390/1" value="30p/50V"/>
-<part name="C10" library="Capacitors" deviceset="C0603C300J5GACTU" device="" package3d_urn="urn:adsk.eagle:package:25020390/1" value="30p/50V"/>
+<part name="Y1" library="Crystals" deviceset="MCSJK-7U-16.00-10-10-80-B-10" device="" package3d_urn="urn:adsk.eagle:package:25022963/1" value="16 MHz"/>
+<part name="C9" library="Capacitors" deviceset="C0603C120J5GACTU" device="" package3d_urn="urn:adsk.eagle:package:25020390/1" value="12p/50V"/>
+<part name="C10" library="Capacitors" deviceset="C0603C120J5GACTU" device="" package3d_urn="urn:adsk.eagle:package:25020390/1" value="12p/50V"/>
 <part name="S38" library="Supplies" deviceset="GND" device=""/>
 <part name="S39" library="Supplies" deviceset="GND" device=""/>
-<part name="Y2" library="ICs" deviceset="ABS07AIG-32.768KHZ-1-T" device="" package3d_urn="urn:adsk.eagle:package:25206263/2" value="32.768 kHz"/>
+<part name="Y2" library="Crystals" deviceset="ABS07AIG-32.768KHZ-1-T" device="" package3d_urn="urn:adsk.eagle:package:25206263/2" value="32.768 kHz"/>
 <part name="C11" library="Capacitors" deviceset="C0603C200J1GACTU" device="" package3d_urn="urn:adsk.eagle:package:25020390/1" value="20p/50V"/>
 <part name="C12" library="Capacitors" deviceset="C0603C200J1GACTU" device="" package3d_urn="urn:adsk.eagle:package:25020390/1" value="20p/50V"/>
@@
 <part name="IC9" library="ICs" deviceset="TLC5973" device="" package3d_urn="urn:adsk.eagle:package:25040621/2" value="TLC5973"/>
 <part name="IC10" library="ICs" deviceset="TLC5973" device="" package3d_urn="urn:adsk.eagle:package:25040621/2" value="TLC5973"/>
-<part name="LED1" library="Diodes" deviceset="CLX6E-FKC" device="" package3d_urn="urn:adsk.eagle:package:25332398/2" value="CLX6E-FKC"/>
-<part name="LED2" library="Diodes" deviceset="CLX6E-FKC" device="" package3d_urn="urn:adsk.eagle:package:25332398/2" value="CLX6E-FKC"/>
-<part name="LED3" library="Diodes" deviceset="CLX6E-FKC" device="" package3d_urn="urn:adsk.eagle:package:25332398/2" value="CLX6E-FKC"/>
-<part name="LED4" library="Diodes" deviceset="CLX6E-FKC" device="" package3d_urn="urn:adsk.eagle:package:25332398/2" value="CLX6E-FKC"/>
+<part name="LED1" library="Diodes" deviceset="CLX6E-FKC" device="" package3d_urn="urn:adsk.eagle:package:25332398/7" value="CLX6E-FKC"/>
+<part name="LED2" library="Diodes" deviceset="CLX6E-FKC" device="" package3d_urn="urn:adsk.eagle:package:25332398/7" value="CLX6E-FKC"/>
+<part name="LED3" library="Diodes" deviceset="CLX6E-FKC" device="" package3d_urn="urn:adsk.eagle:package:25332398/7" value="CLX6E-FKC"/>
+<part name="LED4" library="Diodes" deviceset="CLX6E-FKC" device="" package3d_urn="urn:adsk.eagle:package:25332398/7" value="CLX6E-FKC"/>
 <part name="C5" library="Capacitors" deviceset="C0603C104M5RACTU" device="" package3d_urn="urn:adsk.eagle:package:25020390/1" value="100n/50V"/>
 <part name="C18" library="Capacitors" deviceset="C0603C104M5RACTU" device="" package3d_urn="urn:adsk.eagle:package:25020390/1" value="100n/50V"/>
@@
 <part name="S75" library="Supplies" deviceset="GND" device=""/>
 <part name="S76" library="Supplies" deviceset="GND" device=""/>
+<part name="R21" library="Resistors" deviceset="CRCW06032K00FKEA" device="" package3d_urn="urn:adsk.eagle:package:24925614/1" value="2k/1%"/>
 </parts>
 <sheets>
@@
 <instance part="S76" gate="A" x="-33.02" y="45.72" smashed="yes">
 <attribute name="VALUE" x="-33.02" y="41.148" size="1.27" layer="96" align="bottom-center"/>
+</instance>
+<instance part="R21" gate="A" x="10.16" y="7.62" smashed="yes">
+<attribute name="NAME" x="10.16" y="9.017" size="1.27" layer="95"/>
+<attribute name="VALUE" x="10.16" y="4.953" size="1.27" layer="96"/>
+<attribute name="PARAMETER" x="10.16" y="3.683" size="1.016" layer="96"/>
+<attribute name="PACKAGE" x="12.7" y="7.62" size="1.016" layer="96" align="center"/>
 </instance>
 </instances>
@@
 <segment>
 <pinref part="C10" gate="A" pin="1"/>
-<pinref part="IC14" gate="A" pin="OSC1"/>
 <wire x1="5.08" y1="-5.08" x2="5.08" y2="2.54" width="0.1524" layer="91"/>
 <wire x1="5.08" y1="2.54" x2="5.08" y2="7.62" width="0.1524" layer="91"/>
-<wire x1="5.08" y1="7.62" x2="20.32" y2="7.62" width="0.1524" layer="91"/>
 <pinref part="Y1" gate="A" pin="2"/>
 <wire x1="0" y1="2.54" x2="5.08" y2="2.54" width="0.1524" layer="91"/>
 <junction x="5.08" y="2.54"/>
+<pinref part="R21" gate="A" pin="1"/>
+<wire x1="5.08" y1="7.62" x2="7.62" y2="7.62" width="0.1524" layer="91"/>
 </segment>
 </net>
@@
 </segment>
 </net>
+<net name="N$89" class="0">
+<segment>
+<pinref part="R21" gate="A" pin="2"/>
+<pinref part="IC14" gate="A" pin="OSC1"/>
+<wire x1="17.78" y1="7.62" x2="20.32" y2="7.62" width="0.1524" layer="91"/>
+</segment>
+</net>
