File: NixieClock.sch (EAGLE design)
At the start: 84 parts, among them IC1 SN75468, IC10 TLC5973, IC11 TPS73633DBVT, IC12 MCP111T-300E/TT, IC13 MAX1771ESA+, IC14 TM4C1231H6PMI, IC2 SN75468, IC3 SN75468, IC4 SN75468, IC5 SN74HC595DR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

Commit message: Update
Parts:
- removed IC12: MCP111T-300E/TT, ICs:MCP111T-300E/TT
- C1, C2, C3, C4: value 10n/50V -> 100n/50V; device Capacitors:C0603C103K5RACTU -> Capacitors:C0603C104M5RACTU
- C7: value 10n/50V -> 1u/25V; device Capacitors:C0603C103K5RACTU -> Capacitors:CL10A105KA8NNNC
- IC11: value TPS73633DBVT -> MCP1755T-3302E/DC; device ICs:TPS73633DBVT -> ICs:MCP1755T-3302E/DC
- R1: value 1M/1% -> 100k/1%; device Resistors:CRCW06031M00FKEA -> Resistors:CRCW0603100KFKEA
- R5: value 1M/1% -> 1.5M/1%; device Resistors:CRCW06031M00FKEA -> Resistors:MCPWR12FTEA1504
Connections:
- removed net N$70: C7.1, IC11.NR
- net !JTAG_RST: now also IC11.PWRGD; no longer IC12.OUT
- net 12V: now also IC11.!SHDN, IC11.VIN; no longer IC11.EN, IC11.IN
- net 3V3: now also C7.1, IC11.VOUT; no longer IC11.OUT, IC12.VDD
- net GND: no longer IC12.GND
Other:
- moved on the sheet: C13, C7, C8, D3, IC11, J1, J2, R15

Commit message: Update
Parts:
- removed Q5: BF820, Transistors:BF820
- removed Q6: BF821, Transistors:BF821
- removed R14, R8: 100k/1%, Resistors:CRCW0603100KFKEA
- removed R9: 91k/1%, Resistors:ERJP06F9102V
- added D4: BAS321, Diodes:BAS321
- R16: value 5k/10% -> 5k/20%; device Resistors:T93YB502KT20 -> Resistors:22AR5K
- R17, R18: value 100k/1% -> 10k/1%; device Resistors:CRCW0603100KFKEA -> Resistors:CRCW060310K0FKEA
Connections:
- removed net N$78: Q6.B, R8.2, R9.2
- removed net N$79: Q5.C, R9.1
- removed net N$80: Q5.B, R14.2
- removed net PRE_HV: C14.1, D2.1, Q6.E, R6.2, R8.1
- net DTA_COM: now also D4.1
- net GND: no longer Q5.E
- net HV: now also C14.1, D2.1, R6.2; no longer Q6.C
- net MCU_PWM: no longer R14.1
- net N$68: now also D4.2

Commit message: Update
Parts:
- added C23: 100n/50V, Capacitors:C0603C104M5RACTU
- added C24, C25: 10n/50V, Capacitors:C0603C103K5RACTU
- added R14, R22, R23, R9: 10k/1%, Resistors:CRCW060310K0FKEA
- added R24, R25: 100k/1%, Resistors:CRCW0603100KFKEA
- added R8: 56R/1%, Resistors:CRCW060356R0FKEA
Connections:
- net N$71 renamed CS
- net N$72 renamed SW
- net N$77 renamed REF
- net N$81 renamed FB
- net SW_3 renamed MCU_SW
- removed net LIGHT_SEN: IC14.PE4, J3.5
- removed net SW_1: IC14.PE2, J3.3
- removed net SW_2: IC14.PE1, J3.2
- new net MCU_LS: IC14.PE3, R24.1
- new net MCU_QEA: IC14.PE1, J3.4, R22.1, R9.2
- new net MCU_QEB: IC14.PE2, J3.2, R14.2, R23.1
- new net MCU_VBAT: C23.1, IC14.VBAT, R8.2
- new net N$70: R24.2, R25.1
- new net N$71: J3.5, R25.2
- new net N$72: C24.1, R22.2
- new net N$77: C25.1, R23.2
- net 3V3: now also R14.1, R9.1
- net GND: now also C23.2, C24.2, C25.2, J3.3, M1.7; no longer IC5.!OE, IC6.!OE, IC7.!OE, IC8.!OE, J3.4
- net LED_SDI: now also IC14.PD3; no longer IC14.PA1_U0TX
- net MCU_PWM: now also IC5.!OE, IC6.!OE, IC7.!OE, IC8.!OE
- net SR_RCLK: now also IC14.PA6; no longer IC14.PD1
- net SR_SER: now also IC14.PA5_SSI0TX; no longer IC14.PD0
- net SR_SRCLK: now also IC14.PA2_SSI0CLK; no longer IC14.PD2
- net VBAT: now also R8.1; no longer IC14.VBAT
Other:
- moved on the sheet: C1, C10, C2, C3, C4, C6, C9, J3, R1, Y1

Commit message: Update
Parts:
- added R26: 10k/1%, Resistors:CRCW060310K0FKEA
Connections:
- removed net N$71 (its old number): J3.5, R25.2
- removed net N$72: C24.1, R22.2
- removed net N$77: C25.1, R23.2
- new net QEA_RAW: J3.4, R22.2, R9.1
- new net QEB_RAW: J3.2, R14.1, R23.2
- net 3V3: now also R14.2, R24.1, R26.2, R9.2; no longer R14.1, R9.1
- net GND: now also C24.1, C25.1; no longer C24.2, C25.2
- net MCU_LS: now also J3.5, R25.2; no longer R24.1
- net MCU_PWM: now also R26.1
- net MCU_QEA: now also C24.2; no longer J3.4, R9.2
- net MCU_QEB: now also C25.2; no longer J3.2, R14.2
Other:
- moved on the sheet: C24, C25, R14, R22, R23, R24, R25, R9
