File: NixieClock.brd (EAGLE design)
At the start: 160 x 60 mm, 65 parts, among them IC1 SN75468D, IC10 SN74HC595PW, IC11 TPS73633DBVT, IC12 MCP111T-300E/TT, IC13 MAX1771ESA+, IC2 SN75468D, IC3 SN75468D, IC4 SN75468D, IC5 SN74HC595PW, IC6 SN74HC595PW, IC7 SN74HC595PW, IC8 SN74HC595PW, IC9 SN75468D, J1 PCB Terminal, J2 PCB Terminal, J3 501568-0607, M1 JTAG-10PIN-ARM-CONN, Q1 NIXIE-IN-8-2, Q2 NIXIE-IN-8-2, Q3 NIXIE-IN-8-2, Q4 NIXIE-IN-8-2, Q5 BF722, Q6 BF723, Q7 FQD16N25CTM, U1 TM4C1231H6PMI7, Y1 16 MHz, Y2 32.768 kHz

Commit message: Update
Parts:
- Y2: device ICs:OSCL550P840X380X250-4N -> ICs:OSCCC320X150X90N
- moved R10 220.7 mm to (119.0, 50.0), turned to 90 degrees
- moved J3 205.9 mm to (151.7, 9.40)
- moved C9 172.2 mm to (52.4, 16.4)
- moved R4 152.7 mm to (59.5, 6.20), turned to 270 degrees
- moved R3 148.7 mm to (61.5, 6.20), turned to 270 degrees
- moved C7 146.4 mm to (23.9, 5.10), turned to 90 degrees
- moved R15 140.7 mm to (28.8, 7.80)
- moved C8 139.9 mm to (19.9, 7.80)
- moved C12 135.7 mm to (54.4, 10.1)
- moved IC11 133.3 mm to (19.9, 5.00)
- moved C11 131.9 mm to (54.4, 7.70)
- moved IC12 127.3 mm to (28.8, 4.90)
- moved Y1 122.8 mm to (52.4, 13.6), turned to 90 degrees
- moved C10 122.7 mm to (54.9, 12.9), turned to 90 degrees
- moved R11 122.2 mm to (97.0, 50.0), turned to 90 degrees
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Connections:
- net XOSC0: now also Y2.2; no longer Y2.4

Commit message: Update
Parts:
- C1, C16, C2, C3, C4, C5, C7: value 10u/25V -> 10n/50V; device Capacitors:CAPC3216X170N -> Capacitors:CAPC1608X80N
- moved R5 194.4 mm to (85.5, 26.0), turned to 90 degrees
- moved IC8 186.1 mm to (76.0, 7.00), turned to 270 degrees
- moved IC1 185.4 mm to (109.0, 16.0), turned to 90 degrees
- moved IC2 184.6 mm to (98.0, 16.0), turned to 90 degrees
- moved C1 184.4 mm to (113.2, 4.00)
- moved IC3 183.7 mm to (87.0, 16.0), turned to 90 degrees
- moved C2 182.5 mm to (102.2, 4.00)
- moved IC7 182.2 mm to (87.0, 7.00), turned to 270 degrees
- moved C3 180.7 mm to (91.2, 4.00)
- moved C4 178.9 mm to (80.2, 4.00)
- moved IC6 178.2 mm to (98.0, 7.00), turned to 270 degrees
- moved C5 177.1 mm to (69.2, 4.00)
- moved IC5 174.3 mm to (109.0, 7.00), turned to 270 degrees
- moved R1 166.4 mm to (45.9, 4.40)
- moved D1 159.3 mm to (87.9, 26.9), turned to 90 degrees
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Routing:
- net VSUPP: track 0.00 -> 5.00 mm
- net GND: track 0.00 -> 5.00 mm

Commit message: Update
Parts:
- removed C5: 10n/50V, Capacitors:CAPC1608X80N
- removed IC10: SN74HC595PW, ICs:SOP65P640X120-16N
- removed IC9: SN75468D, ICs:SOIC127P600X175-16N
- added Q8: BF820, Transistors:SOT95P230X110-3N
- added R17, R18: 100k/1%, Resistors:RESC1608X50N
- C16: value 10n/50V -> 10u/25V; device Capacitors:CAPC1608X80N -> Capacitors:CAPC3216X170N
- Q5: value BF722 -> BF820; device Transistors:SOT230P700X180-4N -> Transistors:SOT95P230X110-3N
- Q6: value BF723 -> BF821; device Transistors:SOT230P700X180-4N -> Transistors:SOT95P230X110-3N
- moved J3 82.2 mm to (71.7, -9.60)
- moved PS1 32.7 mm to (126.0, 18.0)
- moved Q5 25.8 mm to (4.40, 39.9), turned to 270 degrees
- moved R10 23.1 mm to (99.0, 47.0)
- moved R11 23.1 mm to (77.0, 47.0)
- moved R12 23.1 mm to (45.0, 47.0)
- moved R13 23.1 mm to (23.0, 47.0)
- moved D1 22.1 mm to (71.0, 41.0)
- moved R5 21.9 mm to (68.7, 40.0)
- moved R14 20.7 mm to (28.8, 13.8), turned to 180 degrees
- moved C1 18.0 mm to (95.2, 3.70)
- moved C2 18.0 mm to (84.2, 3.70)
- moved C3 18.0 mm to (73.2, 3.70)
- moved C4 18.0 mm to (62.2, 3.70)
- moved IC5 18.0 mm to (91.0, 6.70)
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Connections:
- net U1_VDDC renamed MCU_VDDC
- removed net N$27 (its old number): IC4.3, IC8.2
- removed net N$34 (its old number): IC1.14, Q1.2
- removed net N$47 (its old number): IC2.14, Q2.6
- removed net N$69: IC4.10, Q4.9
- new net N$12: IC1.13, Q2.1
- new net N$20: IC2.13, Q2.9
- new net N$28: IC2.3, IC6.4
- new net N$42: IC4.11, Q4.4
- net 3V3: no longer C5.1, IC10.10, IC10.16
- net DTA_COM: no longer IC9.9
- net GND: now also Q5.2, Q8.2, R17.2; no longer C5.2, IC10.13, IC10.8, IC9.2, IC9.3, IC9.4, IC9.5, IC9.6, IC9.7, IC9.8, Q5.3
- net HV: now also Q6.3; no longer Q6.2, Q6.4
- net N$1: now also IC1.7; no longer IC1.1
- net N$10: now also IC1.11, Q1.2; no longer IC2.2, IC6.1
- net N$11: now also IC1.12, Q1.11; no longer IC2.3, IC6.2
- net N$13: now also IC1.14, Q2.2; no longer IC2.5, IC6.4
- net N$14: now also IC1.15, Q2.3; no longer IC2.6, IC6.5
- net N$15: now also IC1.16, Q2.4; no longer IC2.7, IC6.6
- net N$17: now also IC2.10, Q2.5; no longer IC3.1, IC7.15
- net N$18: now also IC2.11, Q2.6; no longer IC3.2, IC7.1
- net N$19: now also IC2.12, Q2.7; no longer IC3.3, IC7.2
- net N$2: now also IC1.6; no longer IC1.2
- net N$21: now also IC2.14, Q2.10; no longer IC3.5, IC7.4
- net N$22: now also IC2.15, Q2.11; no longer IC3.6, IC7.5
- net N$23: now also IC2.7, IC6.15; no longer IC3.7, IC7.6
- net N$25: now also IC2.6, IC6.1; no longer IC4.1, IC8.15
- net N$26: now also IC2.5, IC6.2; no longer IC4.2, IC8.1
- net N$29: now also IC2.2, IC6.5; no longer IC4.5, IC8.4
- net N$3: now also IC1.5; no longer IC1.3
- net N$30: now also IC2.1, IC6.6; no longer IC4.6, IC8.5
- net N$31: now also IC3.7, IC7.15; no longer IC4.7, IC8.6
- net N$32: now also IC3.6, IC7.1; no longer IC1.16, Q1.11
- net N$33: now also IC3.5, IC7.2; no longer IC1.15, Q1.1
- net N$35: now also IC3.3, IC7.4; no longer IC1.13, Q2.11
- net N$36: now also IC3.2, IC7.5; no longer IC1.12, Q2.1
- net N$37: now also IC3.1, IC7.6; no longer IC1.11, Q2.2
- net N$38: now also IC8.7, R18.1; no longer IC9.16, Q4.10
- net N$44: now also IC4.7, IC8.15; no longer IC1.10, Q2.3
- net N$45: now also IC4.6, IC8.1; no longer IC2.16, Q2.4
- net N$46: now also IC4.5, IC8.2; no longer IC2.15, Q2.5
- net N$48: now also IC4.3, IC8.4; no longer IC2.13, Q2.7
- net N$49: now also IC4.2, IC8.5; no longer IC2.12, Q2.9
- net N$5: now also IC1.3; no longer IC1.5
- net N$50: now also IC4.1, IC8.6; no longer IC2.11, Q2.10
- net N$51: now also IC2.16, Q3.1; no longer IC2.10, Q3.11
- net N$52: now also IC3.10, Q3.2; no longer IC3.16, Q3.1
- net N$53: now also IC3.11, Q3.3; no longer IC3.15, Q3.2
- net N$54: now also IC3.12, Q3.4; no longer IC3.14, Q3.3
- net N$57: now also Q3.5; no longer Q3.4
- net N$58: now also IC3.14, Q3.11; no longer IC3.12, Q3.5
- net N$59: now also IC3.15, Q4.1; no longer IC3.11, Q4.11
- net N$6: now also IC1.2; no longer IC1.6
- net N$60: now also IC3.16, Q4.2; no longer IC3.10, Q4.1
- net N$61: now also IC4.10, Q4.3; no longer IC4.16, Q4.2
- net N$62: now also IC4.12, Q4.5; no longer IC4.15, Q4.3
- net N$63: now also IC4.13, Q4.6; no longer IC4.14, Q4.4
- net N$64: now also IC4.14, Q4.7; no longer IC4.13, Q4.5
- net N$65: now also Q8.1, R17.1, R18.2; no longer IC10.14, IC8.9
- net N$66: now also IC4.15, Q4.9; no longer IC10.15, IC9.1
- net N$67: now also IC4.16, Q4.10; no longer IC4.12, Q4.6
- net N$68: now also Q4.11, Q8.3; no longer IC4.11, Q4.7
- net N$7: now also IC1.1; no longer IC1.7
- net N$79: now also Q5.3; no longer Q5.2, Q5.4
- net N$9: now also IC1.10, Q1.1; no longer IC2.1, IC6.15
- net PRE_HV: now also Q6.2; no longer Q6.3
- net SR_RCLK: no longer IC10.12
- net SR_SRCLK: no longer IC10.11
Routing:
- net 3V3: track 0.00 -> 137.6 mm, vias 0 -> 2
- net HV: track 0.00 -> 100.6 mm
- net VBAT: track 0.00 -> 87.5 mm, vias 0 -> 2
- net DTA_COM: track 0.00 -> 80.6 mm, vias 0 -> 5
- net GND: track 5.00 -> 58.7 mm, vias 0 -> 20
- net N$80: track 0.00 -> 52.9 mm, vias 0 -> 2
- net N$59: track 0.00 -> 47.8 mm
- net N$60: track 0.00 -> 44.0 mm
- net N$68: track 0.00 -> 43.3 mm
- net N$67: track 0.00 -> 43.2 mm, vias 0 -> 1
- net N$9: track 0.00 -> 41.0 mm
- net N$66: track 0.00 -> 40.7 mm, vias 0 -> 1
- net N$58: track 0.00 -> 40.4 mm
- net N$61: track 0.00 -> 39.2 mm
- net N$10: track 0.00 -> 37.4 mm
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- added copper zone on layer 1, net 12V
- added copper zone on layer 1, net GND
- added copper zone on layer 1, net N$72
- added copper zone on layer 1, net VSUPP
Other:
- board size 160 x 60 mm -> 138 x 60 mm

Commit message: Update
Parts:
- added MT1, MT2, MT3, MT4: MOUNTING_HOLE_3MM, Misc:MOUNTING_HOLE_3MM
- J1, J2: device Connectors:PCB_TERMINAL_2.8X0.81_RGIHT_ANGLE -> Connectors:PCB_TERMINAL_PAD
- moved J3 37.2 mm to (103.7, 9.40), turned to 180 degrees
- moved PS1 9.06 mm to (117.0, 19.0)
- moved J2 5.91 mm to (3.00, 9.50)
- moved J1 5.47 mm to (3.00, 13.0)
- moved R10 4.59 mm to (103.0, 44.8)
- moved R11 4.59 mm to (81.0, 44.8)
- moved R12 4.59 mm to (49.0, 44.8)
- moved R13 4.59 mm to (27.0, 44.8)
- moved D3 1.20 mm to (4.00, 19.0)
- moved C1 1.00 mm to (95.2, 4.70)
- moved C10 1.00 mm to (48.5, 16.0)
- moved C11 1.00 mm to (50.5, 9.65)
- moved C12 1.00 mm to (50.5, 7.05)
- moved C13 1.00 mm to (11.7, 20.4)
- moved C14 1.00 mm to (17.3, 41.5)
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Connections:
- net N$39 renamed SW_3
- net N$40 renamed SW_2
- net N$41 renamed SW_1
- net N$43 renamed LIGHT_SEN
- net GND: now also MT1.0, MT1.1, MT1.2, MT1.3, MT1.4, MT1.5, MT1.6, MT1.7, MT1.8, MT2.0, MT2.1, MT2.2, MT2.3, MT2.4, MT2.5, MT2.6, MT2.7, MT2.8, MT3.0, MT3.1, MT3.2, MT3.3, MT3.4, MT3.5, MT3.6, MT3.7, MT3.8, MT4.0, MT4.1, MT4.2, MT4.3, MT4.4, MT4.5, MT4.6, MT4.7, MT4.8; no longer J2.2
- net VSUPP: no longer J1.2
Routing:
- net SR_SRCLK: track 0.00 -> 82.4 mm, vias 0 -> 6
- net SR_RCLK: track 0.00 -> 74.7 mm, vias 0 -> 5
- net LIGHT_SEN: track 10.5 -> 84.4 mm
- net SW_1: track 11.4 -> 83.8 mm
- net SW_2: track 11.8 -> 81.1 mm
- net SR_SER: track 0.00 -> 67.5 mm, vias 0 -> 2
- net SW_3: track 12.5 -> 78.5 mm
- net N$16: track 0.00 -> 13.1 mm, vias 0 -> 2
- net N$8: track 0.00 -> 13.0 mm, vias 0 -> 2
- net N$24: track 0.00 -> 13.0 mm, vias 0 -> 2
- net GND: track 58.7 -> 65.6 mm, vias 20 -> 31
- net VBAT: track 87.5 -> 80.8 mm
- net N$76: track 8.36 -> 3.01 mm
- net N$75: track 8.36 -> 3.01 mm
- net N$74: track 8.36 -> 3.01 mm
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- added copper zone on layer 16, net GND
Other:
- board size 138 x 60 mm -> 129 x 50 mm

Commit message: Update
Parts:
- IC5, IC6, IC7, IC8: value SN74HC595PW -> SN74HC595DR; device ICs:SOP65P640X120-16N -> ICs:SOIC127P600X175-16N
- M1: value JTAG-10PIN-ARM-CONN -> JTAG-ARM-10PIN-PLACEHOLDER; device Connectors:20021521-00010T1LF -> Connectors:JTAG-ARM-10PIN-PLACEHOLDER
- moved M1 24.7 mm to (23.2, 6.50), flipped to the bottom, turned to 0 degrees
- moved R3 18.6 mm to (32.8, 18.2), turned to 180 degrees
- moved R4 17.5 mm to (32.8, 16.8), turned to 180 degrees
- moved MT2 10.0 mm to (133.0, 40.0)
- moved C15 9.28 mm to (22.0, 4.42)
- moved C17 9.28 mm to (12.7, 5.30)
- moved IC13 9.28 mm to (17.4, 5.50)
- moved D2 9.09 mm to (18.0, 24.0)
- moved Q6 9.00 mm to (10.5, 33.9)
- moved PS1 8.94 mm to (125.0, 23.0)
- moved Q7 8.80 mm to (19.5, 14.5)
- moved R8 8.70 mm to (10.5, 31.0)
- moved C14 8.48 mm to (18.0, 33.0), turned to 0 degrees
- moved C13 8.40 mm to (11.5, 12.0)
- moved C16 8.30 mm to (9.50, 6.00), turned to 180 degrees
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Routing:
- net JTAG_TCK: track 13.3 -> 35.9 mm, vias 0 -> 1
- net JTAG_TMS: track 13.5 -> 35.5 mm, vias 0 -> 1
- net DTA_COM: track 78.4 -> 56.5 mm
- net JTAG_TDI: track 9.11 -> 30.8 mm, vias 2 -> 1
- net JTAG_TDO: track 9.69 -> 30.4 mm, vias 2 -> 1
- net 12V: track 31.3 -> 49.8 mm
- net N$80: track 52.0 -> 41.6 mm
- net 3V3: track 140.8 -> 130.5 mm, vias 2 -> 4
- net VBAT: track 80.8 -> 90.6 mm
- net N$68: track 43.3 -> 35.8 mm
- net N$81: track 22.3 -> 29.5 mm
- net N$9: track 41.0 -> 34.5 mm
- net N$10: track 37.4 -> 30.9 mm
- net N$61: track 39.2 -> 32.9 mm, vias 0 -> 1
- net N$60: track 44.0 -> 37.9 mm, vias 0 -> 1
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- removed copper zone on layer 1, net 12V
- removed copper zone on layer 1, net VSUPP
Other:
- board size 129 x 50 mm -> 137 x 44 mm

Commit message: Update
Parts:
- moved PS1 4.12 mm to (121.0, 22.0)
- moved MT2 3.16 mm to (130.0, 41.0)
- moved MT3 3.00 mm to (130.0, 4.00)
- moved MT1 1.00 mm to (4.00, 41.0)
Routing:
- net 3V3: track 130.5 -> 137.3 mm, vias 4 -> 5
- net GND: track 64.7 -> 69.6 mm, vias 35 -> 37
- net VBAT: track 90.6 -> 86.7 mm
- net LIGHT_SEN: track 86.1 -> 87.2 mm
Other:
- board size 137 x 44 mm -> 134 x 45 mm

Commit message: Update
Parts:
- added C18, C5: 100n/50V, Capacitors:CAPC1608X80N
- added IC10, IC9: TLC5973, ICs:SOIC127P600X175-8N
- added LED1, LED2, LED3, LED4: CLX6E-FKC, Diodes:CLX6E-FKC
- added R19, R20: 3k3/1%, Resistors:RESC1608X50N
- moved J3 4.00 mm to (108.2, 9.40)
- moved M1 0.20 mm to (23.0, 6.50)
Connections:
- new net LED_SDI: IC9.6, U1.18
- new net N$39: IC9.1, LED1.3
- new net N$40: IC9.3, LED1.1
- new net N$41: IC9.2, LED1.2
- new net N$43: IC10.1, LED3.3
- new net N$69: IC10.2, LED3.2
- new net N$73: IC10.3, LED3.1
- new net N$82: LED3.4, LED4.3
- new net N$84: LED3.5, LED4.2
- new net N$85: LED3.6, LED4.1
- new net N$86: LED1.4, LED2.3
- new net N$87: LED1.5, LED2.2
- new net N$88: LED1.6, LED2.1
- new net N$90: IC9.7, R20.2
- new net N$91: IC10.7, R19.2
- new net N$93: IC10.6, IC9.5
- net 12V: now also LED2.4, LED2.5, LED2.6, LED4.4, LED4.5, LED4.6
- net 3V3: now also C18.1, C5.1, IC10.8, IC9.8
- net GND: now also C18.2, C5.2, IC10.4, IC9.4, R19.1, R20.1
- net N$51: now also Q3.11; no longer Q3.1
- net N$52: now also IC3.14, Q3.5; no longer IC3.10, Q3.2
- net N$53: now also IC3.13, Q3.4; no longer IC3.11, Q3.3
- net N$54: now also Q3.3; no longer Q3.4
- net N$57: now also IC3.11, Q3.2; no longer IC3.13, Q3.5
- net N$58: now also IC3.10, Q3.1; no longer IC3.14, Q3.11
Routing:
- net 12V: track 49.8 -> 143.8 mm, vias 0 -> 3
- net N$93: track 0.00 -> 59.2 mm, vias 0 -> 2
- net N$85: track 0.00 -> 30.9 mm
- net N$88: track 0.00 -> 29.9 mm
- net N$84: track 0.00 -> 28.5 mm
- net N$87: track 0.00 -> 27.8 mm
- net N$82: track 0.00 -> 26.1 mm
- net N$86: track 0.00 -> 25.7 mm
- net N$51: track 31.0 -> 40.1 mm
- net N$52: track 26.3 -> 18.8 mm
- net N$58: track 36.0 -> 28.7 mm
- net LIGHT_SEN: track 87.2 -> 92.4 mm
- net SW_1: track 85.6 -> 90.7 mm
- net SW_3: track 80.5 -> 85.6 mm
- net SW_2: track 83.1 -> 88.1 mm
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- added copper zone on layer 16, net 12V
- added copper zone on layer 16, net 12V1

Commit message: Update
Parts:
- C10, C9: value 43p/50V -> 30p/50V
- C11, C12: value 30p/50V -> 20p/50V
- moved R14 32.5 mm to (6.00, 35.0)
- moved C5 21.6 mm to (41.5, 35.5), turned to 90 degrees
- moved R19 20.8 mm to (97.0, 36.0), turned to 270 degrees
- moved C18 18.9 mm to (95.5, 36.0), turned to 90 degrees
- moved R20 18.6 mm to (43.0, 35.5), turned to 270 degrees
- moved IC9 3.04 mm to (43.5, 30.0)
- moved IC10 2.30 mm to (97.5, 29.2)
- moved C17 1.60 mm to (11.7, 4.05), turned to 180 degrees
- moved C16 1.52 mm to (11.0, 6.25)
- moved R16 1.12 mm to (27.8, 20.7)
- moved R3 0.75 mm to (32.8, 17.5)
- moved R4 0.75 mm to (32.8, 16.0)
- moved R18 0.50 mm to (53.3, 17.5)
Routing:
- net 3V3: track 134.8 -> 192.8 mm, vias 3 -> 5
- net N$80: track 41.6 -> 2.09 mm, vias 2 -> 0
- net LED_SDI: track 1.79 -> 38.9 mm, vias 1 -> 2
- net MCU_PWM: track 5.32 -> 41.4 mm, vias 0 -> 2
- net N$40: track 0.00 -> 14.1 mm, vias 0 -> 1
- net N$73: track 0.00 -> 13.6 mm, vias 0 -> 1
- net N$39: track 0.00 -> 13.1 mm, vias 0 -> 1
- net N$41: track 0.00 -> 12.8 mm, vias 0 -> 1
- net N$43: track 0.00 -> 12.7 mm, vias 0 -> 1
- net N$69: track 0.00 -> 12.5 mm, vias 0 -> 1
- net GND: track 69.6 -> 81.1 mm, vias 37 -> 41
- net N$11: track 21.6 -> 28.0 mm
- net N$91: track 0.00 -> 3.32 mm
- net N$81: track 29.5 -> 26.4 mm
- net N$90: track 0.00 -> 2.07 mm
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- removed copper zone on layer 16, net 12V1
