File: NixieClock.brd (EAGLE design)
At the start: 134 x 45 mm, 79 parts, among them IC1 SN75468D, IC10 TLC5973, IC11 TPS73633DBVT, IC12 MCP111T-300E/TT, IC13 MAX1771ESA+, IC2 SN75468D, IC3 SN75468D, IC4 SN75468D, IC5 SN74HC595DR, IC6 SN74HC595DR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

Commit message: Update
Parts:
- added C19, C21: 10n/50V, Capacitors:CAPC1608X80N
- added C20, C22: 100n/50V, Capacitors:CAPC1608X80N
- IC1, IC2, IC3, IC4: value SN75468D -> SN75468
- IC14: value TM4C1231H6PMI7 -> TM4C1231H6PMI
- R2: value 0.05/1% -> 0R05/1%
- moved R7 1.05 mm to (29.2, 14.5)
- renumbered U1 to IC14
Connections:
- net 3V3: now also C19.1, C20.1, C21.1, C22.1
- net GND: now also C19.2, C20.2, C21.2, C22.2
Routing:
- net GND: track 81.1 -> 90.4 mm, vias 41 -> 44
- net 3V3: track 192.8 -> 193.9 mm
- net JTAG_TDI: track 31.0 -> 31.6 mm

Commit message: Update
Parts:
- added R21: 2k/1%, Resistors:RESC1608X50N
- C10, C9: value 30p/50V -> 12p/50V
- Y1: device ICs:OSCCC320X250X100N -> Crystals:OSCCC320X250X100N
- Y2: device ICs:OSCCC320X150X90N -> Crystals:OSCCC320X150X90N
- moved C10 0.78 mm to (49.8, 14.5)
- moved Y1 0.67 mm to (49.8, 11.8)
- moved C9 0.64 mm to (52.2, 11.8)
- moved R1 0.62 mm to (46.8, 3.40)
- moved C22 0.38 mm to (32.1, 11.0)
Connections:
- new net N$89: IC14.41, R21.2
- net OSC1: now also R21.1; no longer IC14.41
Routing:
- net OSC1: track 6.74 -> 3.18 mm
- net N$89: track 0.00 -> 2.43 mm
- net 3V3: track 193.9 -> 191.4 mm
- net !WAKE: track 1.83 -> 2.42 mm
- net GND: track 90.4 -> 89.9 mm

Commit message: Update
Parts:
- removed IC12: MCP111T-300E/TT, ICs:SOT95P240X110-3N
- C1, C2, C3, C4: value 10n/50V -> 100n/50V
- C7: value 10n/50V -> 1u/25V
- IC11: value TPS73633DBVT -> MCP1755T-3302E/DC; device ICs:SOT95P280X145-5N -> ICs:SOT127P700X180-6N
- R1: value 1M/1% -> 100k/1%
- R5: value 1M/1% -> 1.5M/1%; device Resistors:RESC1608X50N -> Resistors:RESC6331X65N
- moved M1 4.95 mm to (19.5, 10.0), turned to 90 degrees
- moved C8 4.54 mm to (24.5, 4.50), turned to 90 degrees
- moved C7 3.92 mm to (29.5, 2.25)
- moved IC11 3.04 mm to (28.8, 7.00), turned to 90 degrees
- moved R15 2.55 mm to (33.0, 3.00), turned to 270 degrees
- moved C20 2.30 mm to (31.5, 13.8)
- moved R5 1.80 mm to (66.7, 36.5)
- moved R7 1.25 mm to (28.2, 13.8), turned to 180 degrees
- moved C22 1.18 mm to (31.5, 12.0), turned to 180 degrees
- moved R2 1.06 mm to (25.2, 11.5)
- moved R16 1.03 mm to (27.5, 21.7)
- moved R3 1.03 mm to (33.8, 17.8)
- moved R4 1.03 mm to (33.8, 16.2)
- moved C6 1.00 mm to (39.0, 17.5)
- moved D1 0.75 mm to (70.0, 35.2)
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Connections:
- removed net N$70: C7.1, IC11.4
- net !JTAG_RST: now also IC11.5; no longer IC12.1
- net 12V: now also IC11.2; no longer IC11.3
- net 3V3: now also C7.1, IC11.4; no longer IC11.5, IC12.3
- net GND: now also IC11.3, IC11.6; no longer IC11.2, IC12.2
Routing:
- net !JTAG_RST: track 30.7 -> 49.1 mm
- net GND: track 89.9 -> 80.9 mm, vias 44 -> 48
- net 3V3: track 191.4 -> 198.9 mm
- net JTAG_TDO: track 30.5 -> 37.4 mm
- net HV: track 97.8 -> 94.0 mm
- net JTAG_TDI: track 31.6 -> 28.1 mm
- net JTAG_TMS: track 35.9 -> 38.4 mm
- net N$70: track 1.92 -> 0.00 mm
- net N$81: track 26.4 -> 27.9 mm, vias 2 -> 0
- net SR_RCLK: track 73.1 -> 74.3 mm
- net SR_SER: track 66.9 -> 67.9 mm
- net MCU_PWM: track 41.4 -> 42.2 mm
- net N$71: track 6.96 -> 7.66 mm
- net MCU_VDDC: track 14.3 -> 13.7 mm
- net SR_SRCLK: track 76.8 -> 77.3 mm

Commit message: Update
Parts:
- removed Q5: BF820, Transistors:SOT95P230X110-3N
- removed Q6: BF821, Transistors:SOT95P230X110-3N
- removed R14, R8: 100k/1%, Resistors:RESC1608X50N
- removed R9: 91k/1%, Resistors:RESC2012X65N
- added D4: BAS321, Diodes:SOD2512X110N
- R16: value 5k/10% -> 5k/20%; device Resistors:T93YB -> Resistors:22A
- R17, R18: value 100k/1% -> 10k/1%
- moved C14 2.00 mm to (20.0, 33.0)
- moved R16 2.00 mm to (27.5, 19.7), turned to 180 degrees
Connections:
- removed net N$78: Q6.1, R8.2, R9.2
- removed net N$79: Q5.3, R9.1
- removed net N$80: Q5.1, R14.2
- removed net PRE_HV: C14.1, D2.1, Q6.2, R6.2, R8.1
- net DTA_COM: now also D4.1
- net GND: no longer Q5.2
- net HV: now also C14.1, D2.1, R6.2; no longer Q6.3
- net MCU_PWM: no longer R14.1
- net N$68: now also D4.2
- net N$81: now also R16.P$1; no longer R16.1
- net N$83: now also R16.P$2, R16.P$3; no longer R16.2, R16.3
Routing:
- net MCU_PWM: track 42.2 -> 0.00 mm, vias 2 -> 0
- net PRE_HV: track 19.7 -> 0.00 mm
- net DTA_COM: track 56.7 -> 70.4 mm, vias 5 -> 6
- net HV: track 94.0 -> 85.2 mm
- net GND: track 80.9 -> 89.6 mm
- net N$78: track 3.87 -> 0.00 mm
- net N$68: track 35.8 -> 39.5 mm
- net N$79: track 3.16 -> 0.00 mm
- net N$80: track 2.09 -> 0.00 mm
- net N$83: track 9.68 -> 7.67 mm

Commit message: Update
Parts:
- added C23: 100n/50V, Capacitors:CAPC1608X80N
- added C24, C25: 10n/50V, Capacitors:CAPC1608X80N
- added R14, R22, R23, R9: 10k/1%, Resistors:RESC1608X50N
- added R24, R25: 100k/1%, Resistors:RESC1608X50N
- added R8: 56R/1%, Resistors:RESC1608X50N
- moved C15 25.0 mm to (19.5, 29.2)
- moved R2 20.7 mm to (15.0, 29.5), turned to 180 degrees
- moved IC13 18.8 mm to (17.5, 24.2), turned to 90 degrees
- moved C17 16.4 mm to (17.8, 19.2), turned to 0 degrees
- moved Q7 14.5 mm to (8.50, 24.0), turned to 180 degrees
- moved D3 14.2 mm to (15.5, 5.50)
- moved C16 13.3 mm to (18.5, 17.2), turned to 0 degrees
- moved D2 12.9 mm to (6.50, 29.8), turned to 180 degrees
- moved J1 10.6 mm to (11.0, 5.50)
- moved J2 10.6 mm to (11.0, 2.50)
- moved C14 10.4 mm to (10.0, 36.0), turned to 90 degrees
- moved C13 9.76 mm to (21.0, 9.75)
- moved R3 9.55 mm to (43.2, 18.8), turned to 90 degrees
- moved L1 9.26 mm to (9.30, 13.9), turned to 180 degrees
- moved R7 8.85 mm to (22.2, 20.2), turned to 90 degrees
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Connections:
- net N$71 renamed CS
- net N$72 renamed SW
- net N$77 renamed REF
- net N$81 renamed FB
- net SW_3 renamed MCU_SW
- removed net LIGHT_SEN: IC14.59, J3.5
- removed net SW_1: IC14.7, J3.3
- removed net SW_2: IC14.8, J3.2
- new net MCU_LS: IC14.6, R24.1
- new net MCU_QEA: IC14.8, J3.4, R22.1, R9.2
- new net MCU_QEB: IC14.7, J3.2, R14.2, R23.1
- new net MCU_VBAT: C23.1, IC14.37, R8.2
- new net N$70: R24.2, R25.1
- new net N$71: J3.5, R25.2
- new net N$72: C24.1, R22.2
- new net N$77: C25.1, R23.2
- net 3V3: now also R14.1, R9.1
- net GND: now also C23.2, C24.2, C25.2, J3.3, M1.07; no longer IC5.13, IC6.13, IC7.13, IC8.13, J3.4
- net LED_SDI: now also IC14.64; no longer IC14.18
- net MCU_PWM: now also IC5.13, IC6.13, IC7.13, IC8.13
- net SR_RCLK: now also IC14.23; no longer IC14.62
- net SR_SER: now also IC14.22; no longer IC14.61
- net SR_SRCLK: now also IC14.19; no longer IC14.63
- net VBAT: now also R8.1; no longer IC14.37
Routing:
- net LIGHT_SEN: track 92.4 -> 0.00 mm, vias 2 -> 0
- net SW_1: track 90.7 -> 0.00 mm, vias 2 -> 0
- net SW_2: track 88.1 -> 0.00 mm, vias 2 -> 0
- net MCU_QEA: track 0.00 -> 87.0 mm, vias 0 -> 2
- net MCU_QEB: track 0.00 -> 86.1 mm, vias 0 -> 2
- net MCU_VBAT: track 0.00 -> 85.7 mm, vias 0 -> 2
- net VBAT: track 87.0 -> 4.27 mm, vias 2 -> 0
- net MCU_PWM: track 0.00 -> 82.1 mm, vias 0 -> 5
- net MCU_LS: track 0.00 -> 74.6 mm, vias 0 -> 2
- net 12V: track 142.9 -> 103.4 mm
- net FB: track 27.7 -> 7.65 mm
- net LED_SDI: track 39.3 -> 21.5 mm
- net JTAG_TCK: track 36.4 -> 18.8 mm
- net JTAG_TMS: track 38.4 -> 21.3 mm
- net N$71: track 0.00 -> 13.6 mm
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- added copper zone on layer 1, net 12V
- added copper zone on layer 1, net HV
