File: NixieClock.brd (EAGLE design)
At the start: 134 x 45 mm, 89 parts, among them IC1 SN75468, IC10 TLC5973, IC11 MCP1755T-3302E/DC, IC13 MAX1771ESA+, IC14 TM4C1231H6PMI, IC2 SN75468, IC3 SN75468, IC4 SN75468, IC5 SN74HC595DR, IC6 SN74HC595DR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

Commit message: Update
Parts:
- added R26: 10k/1%, Resistors:RESC1608X50N
- moved R24 4.00 mm to (102.2, 19.2)
- moved R25 2.75 mm to (106.2, 19.2)
- moved C24 1.25 mm to (110.2, 16.2), turned to 180 degrees
- moved C25 1.25 mm to (110.2, 17.8), turned to 180 degrees
- turned C13 to 325 degrees
- turned R14 to 180 degrees
- turned R22 to 180 degrees
- turned R23 to 180 degrees
- turned R9 to 180 degrees
Connections:
- removed net N$71 (its old number): J3.5, R25.2
- removed net N$72: C24.1, R22.2
- removed net N$77: C25.1, R23.2
- new net QEA_RAW: J3.4, R22.2, R9.1
- new net QEB_RAW: J3.2, R14.1, R23.2
- net 3V3: now also R14.2, R24.1, R26.2, R9.2; no longer R14.1, R9.1
- net GND: now also C24.1, C25.1; no longer C24.2, C25.2
- net MCU_LS: now also J3.5, R25.2; no longer R24.1
- net MCU_PWM: now also R26.1
- net MCU_QEA: now also C24.2; no longer J3.4, R9.2
- net MCU_QEB: now also C25.2; no longer J3.2, R14.2
Routing:
- net MCU_LS: track 74.6 -> 94.6 mm
- net QEA_RAW: track 0.00 -> 13.9 mm
- net N$71 (its old number): track 13.6 -> 0.00 mm
- net QEB_RAW: track 0.00 -> 13.1 mm
- net MCU_QEA: track 87.0 -> 79.4 mm
- net MCU_QEB: track 86.1 -> 79.3 mm
- net 3V3: track 197.9 -> 199.9 mm
- net N$71: track 1.10 -> 2.35 mm
- net MCU_PWM: track 82.1 -> 83.3 mm
- net N$77: track 1.10 -> 0.00 mm
- net N$72: track 1.10 -> 0.00 mm
